File: OTTOtact.sch (KiCad schematic (older format))
At the start: 188 parts, among them IC1 74HC125, IC2 LM3914, J1 USB, J2 Audio, J3 Speaker, J4 gpio_exp2, J5 gpio_exp1, J6 USB_B_Micro, J7 Conn_01x02, M1 FS8205, SW1 SW_Push, SW10 SW_Push, SW11 SW_Push, SW12 SW_Push, SW13 SW_Push, SW14 SW_Push, SW15 SW_Push, SW16 SW_Push, SW17 SW_Push, SW18 SW_Push, SW19 SW_Push, SW2 SW_Push, SW20 SW_Push, SW21 SW_Push, SW22 SW_Push, SW23 SW_Push, SW24 SW_Push, SW25 SW_Push, SW26 SW_Push, SW27 SW_Push, SW28 SW_Push, SW29 SW_Push, SW3 SW_Push, SW30 SW_Push, SW31 SW_Push, SW32 SW_Push, SW33 SW_Push, SW34 SW_Push, SW35 SW_Push, SW36 SW_Push, SW37 SW_Push, SW38 SW_Push, SW39 SW_Push, SW4 SW_Push, SW40 SW_Push, SW41 SW_Push, SW42 SW_Push, SW43 SW_Push, SW44 SW_Push, SW45 SW_Push, SW46 SW_Push, SW47 SW_Push, SW48 SW_Push, SW49 SW_Push, SW5 SW_Push, SW50 SW_Push, SW51 Rotary_Encoder_Switch, SW52 Rotary_Encoder_Switch, SW53 Rotary_Encoder_Switch, SW54 Rotary_Encoder_Switch, SW55 SW_SPDT, SW6 SW_Push, SW7 SW_Push, SW8 SW_Push, SW9 SW_Push, U1 ATmega32U4-MU, U2 LM386, U3 MCP602, U4 TP4056, U5 FS312F-G, U6 MT3608, Y1 16mhz

Commit message: redesigned the whole audio amplifier circuit, now the headphone switch should work
Parts:
- removed C4: 0.1uf, Capacitor_SMD:C_0805_2012Metric_Pad1.15x1.40mm_HandSolder, symbol Device:C_Small
- removed C5, C6: 10uf, Capacitor_Tantalum_SMD:CP_EIA-2012-12_Kemet-R_Pad1.30x1.05mm_HandSolder, symbol Device:CP1_Small
- removed C7: 0.05uf, Capacitor_SMD:C_0805_2012Metric_Pad1.15x1.40mm_HandSolder, symbol Device:C_Small
- removed C8: 220uf, Capacitor_Tantalum_SMD:CP_EIA-2012-12_Kemet-R_Pad1.30x1.05mm_HandSolder, symbol Device:CP1_Small
- removed J2: Audio, Connector_PinHeader_2.54mm:PinHeader_1x02_P2.54mm_Horizontal, symbol Connector_Generic:Conn_01x02
- removed J3: Speaker, Connector_PinHeader_2.54mm:PinHeader_1x02_P2.54mm_Horizontal, symbol Connector_Generic:Conn_01x02
- removed R2, R21: 10K, Resistor_SMD:R_0805_2012Metric_Pad1.15x1.40mm_HandSolder, symbol Device:R_US
- removed RV1: 100K, Potentiometer_SMD:Potentiometer_Vishay_TS53YJ_Vertical, symbol Device:R_POT_US
- removed U2: LM386, Package_DIP:DIP-8_W7.62mm, symbol Amplifier_Audio:LM386
- added C101, C102: 220uf, Capacitor_Tantalum_SMD:CP_EIA-2012-12_Kemet-R_Pad1.30x1.05mm_HandSolder, symbol Device:CP1_Small
- added C103: 1uf, Capacitor_Tantalum_SMD:CP_EIA-2012-12_Kemet-R_Pad1.30x1.05mm_HandSolder, symbol Device:CP1_Small
- added C104, C105: 0.1uf, Capacitor_Tantalum_SMD:CP_EIA-2012-12_Kemet-R_Pad1.30x1.05mm_HandSolder, symbol Device:CP1_Small
- added J101: audio, Connector_PinHeader_2.54mm:PinHeader_1x04_P2.54mm_Vertical, symbol Connector_Generic:Conn_01x04
- added J102: AudioJack4_Switch, Connector_Audio:SJ-4351X-SMT, symbol Connector:AudioJack4_Switch
- added J103: Speaker, Connector_JST:JST_XH_B02B-XH-A_1x02_P2.50mm_Vertical, symbol Connector_Generic:Conn_01x02
- added R101, R102, R103: 1K, Resistor_SMD:R_0805_2012Metric, symbol Device:R_US
- added R104, R105: 100K, Resistor_SMD:R_0805_2012Metric, symbol Device:R_US
- added R106, R107: 10K, Resistor_SMD:R_0805_2012Metric, symbol Device:R_US
- added U101: LM4860, Package_SO:SOIC-16_3.9x9.9mm_P1.27mm, symbol otto:LM4860
Connections:
- net labels added: GND, L, MIC, R
- wire segments 833 -> 848
- no-connect marks 16 -> 20

Commit message: rewired atmega
Parts:
- Y1: footprint Crystal:Crystal_SMD_5032-2Pin_5.0x3.2mm_HandSoldering -> Crystal:Crystal_SMD_5032-2Pin_5.0x3.2mm
Changed lines of the file:
@@
 F 0 "Y1" V 1250 1912 50  0000 R CNN
 F 1 "16mhz" V 1205 1912 50  0001 R CNN
-F 2 "Crystal:Crystal_SMD_5032-2Pin_5.0x3.2mm_HandSoldering" H 1250 2000 50  0001 C CNN
+F 2 "Crystal:Crystal_SMD_5032-2Pin_5.0x3.2mm" H 1250 2000 50  0001 C CNN
 F 3 "~" H 1250 2000 50  0001 C CNN
 	1    1250 2000
@@
 U 1 1 5BCFFECE
 P 3600 9150
-F 0 "R106" V 3700 9200 50  0000 L CNN
+F 0 "R106" V 3500 9050 50  0000 L CNN
 F 1 "10K" V 3700 9050 50  0000 L CNN
 F 2 "Resistor_SMD:R_0805_2012Metric" V 3640 9140 50  0001 C CNN
@@
 P 3350 9550
 F 0 "C104" V 3450 9550 50  0000 C CNN
-F 1 "0.1uf" V 3250 9600 50  0000 R CNN
+F 1 "0.1uf" V 3250 9650 50  0000 R CNN
 F 2 "Capacitor_Tantalum_SMD:CP_EIA-2012-12_Kemet-R_Pad1.30x1.05mm_HandSolder" H 3350 9550 50  0001 C CNN
 F 3 "~" H 3350 9550 50  0001 C CNN
@@
 U 1 1 5C8AA55E
 P 3750 8750
-F 0 "R107" V 3850 8800 50  0000 L CNN
-F 1 "10K" V 3850 8650 50  0000 L CNN
+F 0 "R107" V 3650 8650 50  0000 L CNN
+F 1 "10K" V 3850 8700 50  0000 L CNN
 F 2 "Resistor_SMD:R_0805_2012Metric" V 3790 8740 50  0001 C CNN
 F 3 "~" H 3750 8750 50  0001 C CNN
@@
 P 4000 8800
 F 0 "C105" V 4100 8800 50  0000 C CNN
-F 1 "0.1uf" V 3900 8850 50  0000 R CNN
+F 1 "0.1uf" V 3900 8900 50  0000 R CNN
 F 2 "Capacitor_Tantalum_SMD:CP_EIA-2012-12_Kemet-R_Pad1.30x1.05mm_HandSolder" H 4000 8800 50  0001 C CNN
 F 3 "~" H 4000 8800 50  0001 C CNN
@@
 U 1 1 5EA73C98
 P 2400 9100
-F 0 "C102" V 2500 9200 50  0000 C CNN
-F 1 "220uf" V 2500 9100 50  0000 R CNN
+F 0 "C102" V 2500 9100 50  0000 C CNN
+F 1 "220uf" V 2300 9200 50  0000 R CNN
 F 2 "Capacitor_Tantalum_SMD:CP_EIA-2012-12_Kemet-R_Pad1.30x1.05mm_HandSolder" H 2400 9100 50  0001 C CNN
 F 3 "~" H 2400 9100 50  0001 C CNN
@@
 U 1 1 5EE00DD6
 P 2850 8450
-F 0 "R104" V 2950 8400 50  0000 L CNN
+F 0 "R104" V 2950 8350 50  0000 L CNN
 F 1 "100K" V 2750 8350 50  0000 L CNN
 F 2 "Resistor_SMD:R_0805_2012Metric" V 2890 8440 50  0001 C CNN
@@
 Wire Wire Line
 	4250 10050 4250 9950
+Connection ~ 4150 10050
 Wire Bus Line
 	6450 7200 6450 9450
@@
 Wire Bus Line
 	7750 6850 7750 9450
-Connection ~ 4150 10050
 $EndSCHEMATC

Commit message: annotation changes - preliminary BOM added
Parts:
- C1: renamed from C14; value 0.1uf -> 0.1uF; footprint Capacitor_SMD:C_0805_2012Metric_Pad1.15x1.40mm_HandSolder -> Capacitor_SMD:C_0805_2012Metric; MFR (none) -> -; MPN (none) -> -; SPN (none) -> -; SPR (none) -> -; SPURL (none) -> -
- C10: renamed from C12; value 100n -> 0.1uF; footprint Capacitor_SMD:C_0805_2012Metric_Pad1.15x1.40mm_HandSolder -> Capacitor_SMD:C_0805_2012Metric; MFR (none) -> -; MPN (none) -> -; SPN (none) -> -; SPR (none) -> -; SPURL (none) -> -
- C11: renamed from C13; value 100n -> 0.1uF; footprint Capacitor_SMD:C_0805_2012Metric_Pad1.15x1.40mm_HandSolder -> Capacitor_SMD:C_0805_2012Metric; MFR (none) -> -; MPN (none) -> -; SPN (none) -> -; SPR (none) -> -; SPURL (none) -> -
- C12: renamed from C15; value 10u -> 10uF; footprint Capacitor_SMD:C_0603_1608Metric_Pad1.05x0.95mm_HandSolder -> Capacitor_SMD:C_0805_2012Metric; MFR (none) -> -; MPN (none) -> -; SPN (none) -> -; SPR (none) -> -; SPURL (none) -> -
- C13: renamed from C16; value 0.1u -> 0.1uF; footprint Capacitor_SMD:C_0603_1608Metric_Pad1.05x0.95mm_HandSolder -> Capacitor_SMD:C_0805_2012Metric; MFR (none) -> -; MPN (none) -> -; SPN (none) -> -; SPR (none) -> -; SPURL (none) -> -
- C14: renamed from C17; footprint Capacitor_SMD:C_0603_1608Metric_Pad1.05x0.95mm_HandSolder -> Capacitor_SMD:C_0805_2012Metric; MFR (none) -> -; MPN (none) -> -; SPN (none) -> -; SPR (none) -> -; SPURL (none) -> -
- C15: renamed from C18; footprint Capacitor_SMD:C_0603_1608Metric_Pad1.05x0.95mm_HandSolder -> Capacitor_Tantalum_SMD:CP_EIA-2012-12_Kemet-R; MFR (none) -> -; MPN (none) -> -; SPN (none) -> -; SPR (none) -> -; SPURL (none) -> -
- C16: renamed from C101; footprint Capacitor_Tantalum_SMD:CP_EIA-2012-12_Kemet-R_Pad1.30x1.05mm_HandSolder -> Capacitor_Tantalum_SMD:CP_EIA-2012-12_Kemet-R; MFR (none) -> -; MPN (none) -> -; SPN (none) -> -; SPR (none) -> -; SPURL (none) -> -
- C17: renamed from C102; footprint Capacitor_Tantalum_SMD:CP_EIA-2012-12_Kemet-R_Pad1.30x1.05mm_HandSolder -> Capacitor_Tantalum_SMD:CP_EIA-2012-12_Kemet-R; MFR (none) -> -; MPN (none) -> -; SPN (none) -> -; SPR (none) -> -; SPURL (none) -> -
- C18: renamed from C103; footprint Capacitor_Tantalum_SMD:CP_EIA-2012-12_Kemet-R_Pad1.30x1.05mm_HandSolder -> Capacitor_Tantalum_SMD:CP_EIA-2012-12_Kemet-R; MFR (none) -> -; MPN (none) -> -; SPN (none) -> -; SPR (none) -> -; SPURL (none) -> -
- C19: renamed from C104; footprint Capacitor_Tantalum_SMD:CP_EIA-2012-12_Kemet-R_Pad1.30x1.05mm_HandSolder -> Capacitor_Tantalum_SMD:CP_EIA-2012-12_Kemet-R; MFR (none) -> -; MPN (none) -> -; SPN (none) -> -; SPR (none) -> -; SPURL (none) -> -
- C2: renamed from C1; value 1uf -> 1uF; footprint Capacitor_SMD:C_0805_2012Metric_Pad1.15x1.40mm_HandSolder -> Capacitor_SMD:C_0805_2012Metric; MFR (none) -> -; MPN (none) -> -; SPN (none) -> -; SPR (none) -> -; SPURL (none) -> -
- C20: renamed from C105; footprint Capacitor_Tantalum_SMD:CP_EIA-2012-12_Kemet-R_Pad1.30x1.05mm_HandSolder -> Capacitor_Tantalum_SMD:CP_EIA-2012-12_Kemet-R; MFR (none) -> -; MPN (none) -> -; SPN (none) -> -; SPR (none) -> -; SPURL (none) -> -
- C3: renamed from C2; value 22pf -> 22pF; footprint Capacitor_SMD:C_0805_2012Metric_Pad1.15x1.40mm_HandSolder -> Capacitor_SMD:C_0805_2012Metric; MFR (none) -> -; MPN (none) -> -; SPN (none) -> -; SPR (none) -> -; SPURL (none) -> -
- C4: renamed from C3; value 22pf -> 22pF; footprint Capacitor_SMD:C_0805_2012Metric_Pad1.15x1.40mm_HandSolder -> Capacitor_SMD:C_0805_2012Metric; MFR (none) -> -; MPN (none) -> -; SPN (none) -> -; SPR (none) -> -; SPURL (none) -> -
- C5: renamed from C19; value 0.1uf -> 0.1uF; footprint Capacitor_SMD:C_0805_2012Metric_Pad1.15x1.40mm_HandSolder -> Capacitor_SMD:C_0805_2012Metric; MFR (none) -> -; MPN (none) -> -; SPN (none) -> -; SPR (none) -> -; SPURL (none) -> -
- C6: renamed from C21; value 0.1uf -> 0.1uF; footprint Capacitor_SMD:C_0805_2012Metric_Pad1.15x1.40mm_HandSolder -> Capacitor_SMD:C_0805_2012Metric; MFR (none) -> -; MPN (none) -> -; SPN (none) -> -; SPR (none) -> -; SPURL (none) -> -
- C7: renamed from C9; value 100n -> 0.1uF; footprint Capacitor_SMD:C_0805_2012Metric_Pad1.15x1.40mm_HandSolder -> Capacitor_SMD:C_0805_2012Metric; MFR (none) -> -; MPN (none) -> -; SPN (none) -> -; SPR (none) -> -; SPURL (none) -> -
- C8: renamed from C10; value 100n -> 0.1uF; footprint Capacitor_SMD:C_0805_2012Metric_Pad1.15x1.40mm_HandSolder -> Capacitor_SMD:C_0805_2012Metric; MFR (none) -> -; MPN (none) -> -; SPN (none) -> -; SPR (none) -> -; SPURL (none) -> -
- C9: renamed from C11; value 100n -> 0.1uF; footprint Capacitor_SMD:C_0805_2012Metric_Pad1.15x1.40mm_HandSolder -> Capacitor_SMD:C_0805_2012Metric; MFR (none) -> -; MPN (none) -> -; SPN (none) -> -; SPR (none) -> -; SPURL (none) -> -
- D1: footprint LED_SMD:LED_0805_2012Metric_Pad1.15x1.40mm_HandSolder -> LED_SMD:LED_0805_2012Metric; MFR (none) -> -; MPN (none) -> HSMW-C170-U0000; SPN (none) -> -; SPR (none) -> -; SPURL (none) -> -
- D10, D11, D12, D13, D14, D15, D16, D17, D18, D19, D2, D20, D21, D22, D23, D24, D25, D26, D27, D28, D29, D3, D30, D31, D32, D33, D34, D35, D36, D37, D38, D39, D4, D40, D41, D42, D43, D44, D45, D46, D47, D48, D49, D5, D50, D51, D52, D53, D54, D55, D6, D7, D8, D9: MFR (none) -> -; MPN (none) -> 1N4148W-E3-18; SPN (none) -> 78-1N4148W-E3-18; SPR (none) -> mouser; SPURL (none) -> -
- D56: footprint LED_SMD:LED_0603_1608Metric -> LED_SMD:LED_0805_2012Metric; MFR (none) -> -; MPN (none) -> HSMC-C170-T0000; SPN (none) -> -; SPR (none) -> -; SPURL (none) -> -
- D57: footprint LED_SMD:LED_0603_1608Metric -> LED_SMD:LED_0805_2012Metric; MFR (none) -> -; MPN (none) -> HSMQ-C170-T0000; SPN (none) -> -; SPR (none) -> -; SPURL (none) -> -
- D58: footprint Diode_SMD:D_SMC_Handsoldering -> Diode_SMD:D_SMC; MFR (none) -> -; MPN (none) -> SS34; SPN (none) -> 512-SS34; SPR (none) -> mouser; SPURL (none) -> -
- D59, D60, D61, D62, D63: footprint LED_SMD:LED_0603_1608Metric -> LED_SMD:LED_0805_2012Metric; MFR (none) -> -; MPN (none) -> HSMW-C170-U0000; SPN (none) -> -; SPR (none) -> -; SPURL (none) -> -
- IC1: MFR (none) -> -; MPN (none) -> SN74HC125DR; SPN (none) -> 595-SN74HC125DR; SPR (none) -> -; SPURL (none) -> -
- IC2: MFR (none) -> -; MPN (none) -> LM3914VX/NOPB; SPN (none) -> 926-LM3914VX/NOPB; SPR (none) -> mouser; SPURL (none) -> -
- J1: MFR (none) -> -; MPN (none) -> 1x04 pin header; SPN (none) -> -; SPR (none) -> -; SPURL (none) -> -
- J2: renamed from J6; MFR (none) -> Molex; MPN (none) -> 105017-0001; SPN (none) -> 538-105017-0001; SPR (none) -> mouser; SPURL (none) -> -
- J3: renamed from J7; value Conn_01x02 -> battery; MFR (none) -> JST; MPN (none) -> XH-B02B; SPN (none) -> -; SPR (none) -> -; SPURL (none) -> -
- J4: renamed from J101; MFR (none) -> -; MPN (none) -> 1x04 pin header; SPN (none) -> -; SPR (none) -> -; SPURL (none) -> -
- J5: renamed from J102; value AudioJack4_Switch -> SJ1-42536-SMT; MFR (none) -> Cui; MPN (none) -> SJ1-42536-SMT; SPN (none) -> 490-SJ1-42536-SMT-TR; SPR (none) -> mouser; SPURL (none) -> -
- J6: renamed from J103; MFR (none) -> JST; MPN (none) -> XH-B02B; SPN (none) -> -; SPR (none) -> -; SPURL (none) -> -
- J7: renamed from J4; MFR (none) -> 2x20 pin header; MPN (none) -> -; SPN (none) -> -; SPR (none) -> -; SPURL (none) -> -
- J8: renamed from J5; MFR (none) -> 2x20 long pin header; MPN (none) -> -; SPN (none) -> -; SPR (none) -> -; SPURL (none) -> -
- JP1, SW1, SW10, SW11, SW12, SW13, SW14, SW15, SW16, SW17, SW18, SW19, SW2, SW20, SW21, SW22, SW23, SW24, SW25, SW26, SW27, SW28, SW29, SW3, SW30, SW31, SW32, SW33, SW34, SW35, SW36, SW37, SW38, SW39, SW4, SW40, SW41, SW42, SW43, SW44, SW45, SW46, SW47, SW48, SW49, SW5, SW50, SW6, SW7, SW8, SW9: MFR (none) -> -; MPN (none) -> -; SPN (none) -> -; SPR (none) -> -; SPURL (none) -> -
- L1: MFR (none) -> Epcos; MPN (none) -> B82472G6223M000; SPN (none) -> 871-B82472G6223M000; SPR (none) -> mouser; SPURL (none) -> -
- M1: MFR (none) -> -; MPN (none) -> FS8205 SOT-23; SPN (none) -> -; SPR (none) -> -; SPURL (none) -> -
- R1: footprint Resistor_SMD:R_0805_2012Metric_Pad1.15x1.40mm_HandSolder -> Resistor_SMD:R_0805_2012Metric; MFR (none) -> -; MPN (none) -> -; SPN (none) -> -; SPR (none) -> -; SPURL (none) -> -
- R10: renamed from R11; footprint Resistor_SMD:R_0805_2012Metric_Pad1.15x1.40mm_HandSolder -> Resistor_SMD:R_0805_2012Metric; MFR (none) -> -; MPN (none) -> -; SPN (none) -> -; SPR (none) -> -; SPURL (none) -> -
- R11: renamed from R12; footprint Resistor_SMD:R_0805_2012Metric_Pad1.15x1.40mm_HandSolder -> Resistor_SMD:R_0805_2012Metric; MFR (none) -> -; MPN (none) -> -; SPN (none) -> -; SPR (none) -> -; SPURL (none) -> -
- R12: renamed from R13; footprint Resistor_SMD:R_0805_2012Metric_Pad1.15x1.40mm_HandSolder -> Resistor_SMD:R_0805_2012Metric; MFR (none) -> -; MPN (none) -> -; SPN (none) -> -; SPR (none) -> -; SPURL (none) -> -
- R13: renamed from R14; footprint Resistor_SMD:R_0805_2012Metric_Pad1.15x1.40mm_HandSolder -> Resistor_SMD:R_0805_2012Metric; MFR (none) -> -; MPN (none) -> -; SPN (none) -> -; SPR (none) -> -; SPURL (none) -> -
- R14: renamed from R15; value 470 -> 470K; footprint Resistor_SMD:R_0805_2012Metric_Pad1.15x1.40mm_HandSolder -> Resistor_SMD:R_0805_2012Metric; MFR (none) -> -; MPN (none) -> -; SPN (none) -> -; SPR (none) -> -; SPURL (none) -> -
- R15: renamed from R16; footprint Resistor_SMD:R_0805_2012Metric_Pad1.15x1.40mm_HandSolder -> Resistor_SMD:R_0805_2012Metric; MFR (none) -> -; MPN (none) -> -; SPN (none) -> -; SPR (none) -> -; SPURL (none) -> -
- R16: renamed from R17; value 820 -> 820K; footprint Resistor_SMD:R_0805_2012Metric_Pad1.15x1.40mm_HandSolder -> Resistor_SMD:R_0805_2012Metric; MFR (none) -> -; MPN (none) -> -; SPN (none) -> -; SPR (none) -> -; SPURL (none) -> -
- R17: renamed from R18; footprint Resistor_SMD:R_0805_2012Metric_Pad1.15x1.40mm_HandSolder -> Resistor_SMD:R_0805_2012Metric; MFR (none) -> -; MPN (none) -> -; SPN (none) -> -; SPR (none) -> -; SPURL (none) -> -
- R18: renamed from R19; footprint Resistor_SMD:R_0805_2012Metric_Pad1.15x1.40mm_HandSolder -> Resistor_SMD:R_0805_2012Metric; MFR (none) -> -; MPN (none) -> -; SPN (none) -> -; SPR (none) -> -; SPURL (none) -> -
- R19: renamed from R20; footprint Resistor_SMD:R_0805_2012Metric_Pad1.15x1.40mm_HandSolder -> Resistor_SMD:R_0805_2012Metric; MFR (none) -> -; MPN (none) -> -; SPN (none) -> -; SPR (none) -> -; SPURL (none) -> -
- R2: renamed from R3; value 330 -> 330K; footprint Resistor_SMD:R_0805_2012Metric_Pad1.15x1.40mm_HandSolder -> Resistor_SMD:R_0805_2012Metric; MFR (none) -> -; MPN (none) -> -; SPN (none) -> -; SPR (none) -> -; SPURL (none) -> -
- R20: renamed from R22; footprint Resistor_SMD:R_0603_1608Metric -> Resistor_SMD:R_0805_2012Metric; MFR (none) -> -; MPN (none) -> -; SPN (none) -> -; SPR (none) -> -; SPURL (none) -> -
- R21: renamed from R24; footprint Resistor_SMD:R_0603_1608Metric -> Resistor_SMD:R_0805_2012Metric; MFR (none) -> -; MPN (none) -> -; SPN (none) -> -; SPR (none) -> -; SPURL (none) -> -
- R22: renamed from R25; footprint Resistor_SMD:R_0603_1608Metric -> Resistor_SMD:R_0805_2012Metric; MFR (none) -> -; MPN (none) -> -; SPN (none) -> -; SPR (none) -> -; SPURL (none) -> -
- R23: renamed from R26; value 100 -> 100K; footprint Resistor_SMD:R_0603_1608Metric -> Resistor_SMD:R_0805_2012Metric; MFR (none) -> -; MPN (none) -> -; SPN (none) -> -; SPR (none) -> -; SPURL (none) -> -
- R24: renamed from R27; footprint Resistor_SMD:R_0603_1608Metric -> Resistor_SMD:R_0805_2012Metric; MFR (none) -> -; MPN (none) -> -; SPN (none) -> -; SPR (none) -> -; SPURL (none) -> -
- R25: renamed from R28; footprint Resistor_SMD:R_0603_1608Metric -> Resistor_SMD:R_0805_2012Metric; MFR (none) -> -; MPN (none) -> -; SPN (none) -> -; SPR (none) -> -; SPURL (none) -> -
- R26: renamed from R29; footprint Resistor_SMD:R_0603_1608Metric -> Resistor_SMD:R_0805_2012Metric; MFR (none) -> -; MPN (none) -> -; SPN (none) -> -; SPR (none) -> -; SPURL (none) -> -
- R27: renamed from R23; footprint Resistor_SMD:R_0603_1608Metric -> Resistor_SMD:R_0805_2012Metric; MFR (none) -> -; MPN (none) -> -; SPN (none) -> -; SPR (none) -> -; SPURL (none) -> -
- R28: renamed from R101; MFR (none) -> -; MPN (none) -> -; SPN (none) -> -; SPR (none) -> -; SPURL (none) -> -
- R29: renamed from R102; MFR (none) -> -; MPN (none) -> -; SPN (none) -> -; SPR (none) -> -; SPURL (none) -> -
- R3: renamed from R4; footprint Resistor_SMD:R_0805_2012Metric_Pad1.15x1.40mm_HandSolder -> Resistor_SMD:R_0805_2012Metric; MFR (none) -> -; MPN (none) -> -; SPN (none) -> -; SPR (none) -> -; SPURL (none) -> -
- R30: renamed from R103; MFR (none) -> -; MPN (none) -> -; SPN (none) -> -; SPR (none) -> -; SPURL (none) -> -
- R31: renamed from R104; MFR (none) -> -; MPN (none) -> -; SPN (none) -> -; SPR (none) -> -; SPURL (none) -> -
- R32: renamed from R105; MFR (none) -> -; MPN (none) -> -; SPN (none) -> -; SPR (none) -> -; SPURL (none) -> -
- R33: renamed from R106; MFR (none) -> -; MPN (none) -> -; SPN (none) -> -; SPR (none) -> -; SPURL (none) -> -
- R34: renamed from R107; MFR (none) -> -; MPN (none) -> -; SPN (none) -> -; SPR (none) -> -; SPURL (none) -> -
- R4: renamed from R5; footprint Resistor_SMD:R_0805_2012Metric_Pad1.15x1.40mm_HandSolder -> Resistor_SMD:R_0805_2012Metric; MFR (none) -> -; MPN (none) -> -; SPN (none) -> -; SPR (none) -> -; SPURL (none) -> -
- R5: renamed from R6; footprint Resistor_SMD:R_0805_2012Metric_Pad1.15x1.40mm_HandSolder -> Resistor_SMD:R_0805_2012Metric; MFR (none) -> -; MPN (none) -> -; SPN (none) -> -; SPR (none) -> -; SPURL (none) -> -
- R6: renamed from R7; footprint Resistor_SMD:R_0805_2012Metric_Pad1.15x1.40mm_HandSolder -> Resistor_SMD:R_0805_2012Metric; MFR (none) -> -; MPN (none) -> -; SPN (none) -> -; SPR (none) -> -; SPURL (none) -> -
- R7: renamed from R8; footprint Resistor_SMD:R_0805_2012Metric_Pad1.15x1.40mm_HandSolder -> Resistor_SMD:R_0805_2012Metric; MFR (none) -> -; MPN (none) -> -; SPN (none) -> -; SPR (none) -> -; SPURL (none) -> -
- R8: renamed from R9; footprint Resistor_SMD:R_0805_2012Metric_Pad1.15x1.40mm_HandSolder -> Resistor_SMD:R_0805_2012Metric; MFR (none) -> -; MPN (none) -> -; SPN (none) -> -; SPR (none) -> -; SPURL (none) -> -
- R9: renamed from R10; footprint Resistor_SMD:R_0805_2012Metric_Pad1.15x1.40mm_HandSolder -> Resistor_SMD:R_0805_2012Metric; MFR (none) -> -; MPN (none) -> -; SPN (none) -> -; SPR (none) -> -; SPURL (none) -> -
- RV1: renamed from RV2; value R_POT_TRIM_US -> 10K; MFR (none) -> -; MPN (none) -> TS53YJ103MR10; SPN (none) -> -; SPR (none) -> -; SPURL (none) -> -
- SW51, SW52, SW53, SW54: MFR (none) -> -; MPN (none) -> EC12D1564404; SPN (none) -> -; SPR (none) -> -; SPURL (none) -> -
- SW55: value SW_SPDT -> ON_OFF_SWITCH; MFR (none) -> E-Switch; MPN (none) -> EG1224; SPN (none) -> 612-EG1224; SPR (none) -> mouser; SPURL (none) -> -
- U1: value ATmega32U4-MU -> ATMEGA32U4-AU; MFR (none) -> -; MPN (none) -> ATMEGA32U4-AU; SPN (none) -> 556-ATMEGA32U4-AU; SPR (none) -> -; SPURL (none) -> -
- U2: renamed from U3; MFR (none) -> -; MPN (none) -> MCP6022T-I/SN; SPN (none) -> -; SPR (none) -> -; SPURL (none) -> -
- U3: renamed from U4; MFR (none) -> -; MPN (none) -> TP4056 SOP-8; SPN (none) -> -; SPR (none) -> -; SPURL (none) -> -
- U4: renamed from U5; footprint Package_TO_SOT_SMD:SOT-23-6_Handsoldering -> Package_TO_SOT_SMD:SOT-23-6; MFR (none) -> -; MPN (none) -> FS312F-G SOT-23; SPN (none) -> -; SPR (none) -> -; SPURL (none) -> -
- U5: renamed from U6; footprint Package_TO_SOT_SMD:SOT-23-6_Handsoldering -> Package_TO_SOT_SMD:SOT-23-6; MFR (none) -> -; MPN (none) -> MT3608 SOT-23; SPN (none) -> -; SPR (none) -> -; SPURL (none) -> -
- U6: renamed from U101; MFR (none) -> -; MPN (none) -> LM4860MX/NOPB; SPN (none) -> -; SPR (none) -> -; SPURL (none) -> -
- Y1: MFR (none) -> -; MPN (none) -> SG5032CCN 16.000000M-HJGA3; SPN (none) -> 581-KC7050A16.C3GE; SPR (none) -> mouser; SPURL (none) -> -
Other:
- moved on the sheet: U1, U2A

Commit message: display footprint, bom update
Parts:
- added J10: Conn_01x04_Male, Connector_JST:JST_SH_SM04B-SRSS-TB_1x04-1MP_P1.00mm_Horizontal, symbol Connector:Conn_01x04_Male
- added U7: CR2013-MI2120, Display:TJCTM24028-SPI, symbol Driver_Display:CR2013-MI2120
- J5: footprint Connector_Audio:SJ-4351X-SMT -> SJ1:CUI_SJ1-42536-SMT
- Y1: footprint Crystal:Crystal_SMD_5032-2Pin_5.0x3.2mm -> Crystal:Crystal_SMD_Abracon_ABM3-2Pin_5.0x3.2mm; MPN SG5032CCN 16.000000M-HJGA3 -> ABM3-16.000MHZ-D2Y-T; SPN 581-KC7050A16.C3GE -> -
Connections:
- wire segments 848 -> 865
- no-connect marks 20 -> 30

Commit message: 0.1v rellease
Parts:
- added C21: 0.1uF, Capacitor_SMD:C_0805_2012Metric, symbol Device:C_Small
- added C22: 0.01uF, Capacitor_SMD:C_0805_2012Metric, symbol Device:C_Small
- added C23: 1uF, Capacitor_SMD:C_0805_2012Metric, symbol Device:C_Small
- added C24: 100pF, Capacitor_SMD:C_0805_2012Metric, symbol Device:C_Small
- added MK1: Microphone, CMA-4544PF-W:CMA-4544PF-W, symbol Device:Microphone
- added Q1: 2N7000, Package_TO_SOT_THT:TO-92_Inline, symbol Transistor_FET:2N7000
- added R35, R41: 100K, Resistor_SMD:R_0805_2012Metric, symbol Device:R_US
- added R36, R38, R40: 1K, Resistor_SMD:R_0805_2012Metric, symbol Device:R_US
- added R37, R39: 1M, Resistor_SMD:R_0805_2012Metric, symbol Device:R_US
- added U8: MAX4466, Package_TO_SOT_SMD:SOT-353_SC-70-5, symbol Amplifier_Audio:MAX4466
- C15, C16, C17: footprint Capacitor_Tantalum_SMD:CP_EIA-2012-12_Kemet-R -> Capacitor_Tantalum_SMD:CP_EIA-3528-21_Kemet-B
- C18: footprint Capacitor_Tantalum_SMD:CP_EIA-2012-12_Kemet-R -> Capacitor_Tantalum_SMD:CP_EIA-3216-18_Kemet-A
- IC2: footprint Package_LCC:PLCC-20 -> Package_DIP:DIP-18_W7.62mm
- J5: footprint SJ1:CUI_SJ1-42536-SMT -> Connector_Audio:PJ-237-6A
- L1: footprint Inductor_SMD:L_7.3x7.3_H4.5 -> Inductor_SMD:L_Wuerth_HCI-1040
- RV1: footprint Potentiometer_SMD:Potentiometer_Vishay_TS53YJ_Vertical -> 3362P-1-103LF:3362P_1
- SW55: footprint Button_Switch_THT:SW_E-Switch_EG1224_SPDT_Angled -> Button_Switch_THT:SK-12E12-G5
- U7: value CR2013-MI2120 -> TJCTM24028-SPI
Connections:
- wire segments 865 -> 893
