File: OTTO-main/OTTO-main.kicad_pcb (KiCad board)
At the start: 2 copper layers, 41 parts, among them IC1 74HC125, U2 STM32F103CBTx, U3 ILI9341, U4 MCP602, Y1 8mhz

Commit message: Revert "added a reset button to the power board"
This reverts commit bbfaa2fb8df27d7f63d1a584e9f51fc8f5fa6fe3.
Parts:
- added C1: 10uf, Capacitor_Tantalum_SMD:CP_EIA-3216-18_Kemet-A, F.Cu at (171.9, 27.4)
- added C2: 22uf, Capacitor_Tantalum_SMD:CP_EIA-3216-18_Kemet-A, F.Cu at (159.4, 27.4)
- added D10: D_ALT, Diode_SMD:D_SOD-123, B.Cu at (255.4, 94.9)
- added D11: D_ALT, Diode_SMD:D_SOD-123, B.Cu at (34.5, 43.6)
- added D12: D_ALT, Diode_SMD:D_SOD-123, B.Cu at (34.5, 59.7)
- added D13: D_ALT, Diode_SMD:D_SOD-123, B.Cu at (34.5, 75.8)
- added D14: D_ALT, Diode_SMD:D_SOD-123, B.Cu at (47.0, 75.8)
- added D15: D_ALT, Diode_SMD:D_SOD-123, B.Cu at (59.6, 75.8)
- added D16: D_ALT, Diode_SMD:D_SOD-123, B.Cu at (72.2, 75.8)
- added D17: D_ALT, Diode_SMD:D_SOD-123, B.Cu at (84.8, 75.8)
- added D18: D_ALT, Diode_SMD:D_SOD-123, B.Cu at (97.5, 75.8)
- added D19: D_ALT, Diode_SMD:D_SOD-123, B.Cu at (110.0, 75.8)
- added D20: D_ALT, Diode_SMD:D_SOD-123, B.Cu at (122.7, 75.8)
- added D21: D_ALT, Diode_SMD:D_SOD-123, B.Cu at (34.5, 91.9)
- added D22: D_ALT, Diode_SMD:D_SOD-123, B.Cu at (47.0, 91.9)
- added D23: D_ALT, Diode_SMD:D_SOD-123, B.Cu at (59.6, 91.9)
- added D24: D_ALT, Diode_SMD:D_SOD-123, B.Cu at (72.2, 91.9)
- added D25: D_ALT, Diode_SMD:D_SOD-123, B.Cu at (84.8, 91.9)
- added D26: D_ALT, Diode_SMD:D_SOD-123, B.Cu at (97.5, 91.9)
- added D27: D_ALT, Diode_SMD:D_SOD-123, B.Cu at (110.0, 91.9)
- added D28: D_ALT, Diode_SMD:D_SOD-123, B.Cu at (122.7, 91.9)
- added D29: D_ALT, Diode_SMD:D_SOD-123, B.Cu at (135.2, 91.9)
- added D30: D_ALT, Diode_SMD:D_SOD-123, B.Cu at (135.2, 75.8)
- added D5: D_ALT, Diode_SMD:D_SOD-123, B.Cu at (242.8, 62.7)
- added D6: D_ALT, Diode_SMD:D_SOD-123, B.Cu at (255.4, 62.7)
- added D7: D_ALT, Diode_SMD:D_SOD-123, B.Cu at (242.8, 78.8)
- added D8: D_ALT, Diode_SMD:D_SOD-123, B.Cu at (255.4, 78.8)
- added D9: D_ALT, Diode_SMD:D_SOD-123, B.Cu at (242.8, 94.9)
- added J1: POWER_BOARD, Connector_PinSocket_2.54mm:PinSocket_1x07_P2.54mm_Vertical, B.Cu at (151.4, 37.0)
- added J2: AUDIO_BOARD, Connector_PinSocket_2.54mm:PinSocket_1x10_P2.54mm_Vertical, B.Cu at (228.2, 68.5)
- added J3: Raspberry_Pi_2_3, Connector_PinHeader_2.54mm:PinHeader_2x20_P2.54mm_Vertical, F.Cu at (102.1, 106.4)
- added J4: MICROPHONE, Connector_PinSocket_2.54mm:PinSocket_1x02_P2.54mm_Vertical, B.Cu at (260.6, 108.0)
- added REF**: MountingHole_3.2mm_M3, MountingHole:MountingHole_3.2mm_M3, F.Cu at (260.4, 38.5)
- added REF**: MountingHole_3.2mm_M3, MountingHole:MountingHole_3.2mm_M3, F.Cu at (144.9, 110.5)
- added REF**: MountingHole_3.2mm_M3, MountingHole:MountingHole_3.2mm_M3, F.Cu at (143.9, 38.5)
- added REF**: MountingHole_3.2mm_M3, MountingHole:MountingHole_3.2mm_M3, F.Cu at (49.0, 38.5)
- added SW1: Rotary_Encoder_Switch, Rotary_Encoder:RotaryEncoder_Alps_EC12E-Switch_Vertical_H20mm_CircularMountingHoles, F.Cu at (53.3, 51.7)
- added SW10: SW_SPST, Button_Switch_THT:Tactile_Switch_12x12x7.3_mm, F.Cu at (255.4, 94.9)
- added SW11: SW_SPST, Button_Switch_THT:Tactile_Switch_12x12x7.3_mm, F.Cu at (34.5, 43.6)
- added SW12: SW_SPST, Button_Switch_THT:Tactile_Switch_12x12x7.3_mm, F.Cu at (34.5, 59.7)
- added SW13: SW_SPST, Button_Switch_THT:Tactile_Switch_12x12x7.3_mm, F.Cu at (34.5, 75.8)
- added SW14: SW_SPST, Button_Switch_THT:Tactile_Switch_12x12x7.3_mm, F.Cu at (47.0, 75.8)
- added SW15: SW_SPST, Button_Switch_THT:Tactile_Switch_12x12x7.3_mm, F.Cu at (59.6, 75.8)
- added SW16: SW_SPST, Button_Switch_THT:Tactile_Switch_12x12x7.3_mm, F.Cu at (72.2, 75.8)
- added SW17: SW_SPST, Button_Switch_THT:Tactile_Switch_12x12x7.3_mm, F.Cu at (84.8, 75.8)
- added SW18: SW_SPST, Button_Switch_THT:Tactile_Switch_12x12x7.3_mm, F.Cu at (97.5, 75.8)
- added SW19: SW_SPST, Button_Switch_THT:Tactile_Switch_12x12x7.3_mm, F.Cu at (110.0, 75.8)
- added SW2: Rotary_Encoder_Switch, Rotary_Encoder:RotaryEncoder_Alps_EC12E-Switch_Vertical_H20mm_CircularMountingHoles, F.Cu at (78.5, 51.7)
- added SW20: SW_SPST, Button_Switch_THT:Tactile_Switch_12x12x7.3_mm, F.Cu at (122.7, 75.8)
- added SW21: SW_SPST, Button_Switch_THT:Tactile_Switch_12x12x7.3_mm, F.Cu at (34.5, 91.9)
- added SW22: SW_SPST, Button_Switch_THT:Tactile_Switch_12x12x7.3_mm, F.Cu at (47.0, 91.9)
- added SW23: SW_SPST, Button_Switch_THT:Tactile_Switch_12x12x7.3_mm, F.Cu at (59.6, 91.9)
- added SW24: SW_SPST, Button_Switch_THT:Tactile_Switch_12x12x7.3_mm, F.Cu at (72.2, 91.9)
- added SW25: SW_SPST, Button_Switch_THT:Tactile_Switch_12x12x7.3_mm, F.Cu at (84.8, 91.9)
- added SW26: SW_SPST, Button_Switch_THT:Tactile_Switch_12x12x7.3_mm, F.Cu at (97.5, 91.9)
- added SW27: SW_SPST, Button_Switch_THT:Tactile_Switch_12x12x7.3_mm, F.Cu at (110.0, 91.9)
- added SW28: SW_SPST, Button_Switch_THT:Tactile_Switch_12x12x7.3_mm, F.Cu at (122.7, 91.9)
- added SW29: SW_SPST, Button_Switch_THT:Tactile_Switch_12x12x7.3_mm, F.Cu at (135.2, 91.9)
- added SW3: Rotary_Encoder_Switch, Rotary_Encoder:RotaryEncoder_Alps_EC12E-Switch_Vertical_H20mm_CircularMountingHoles, F.Cu at (103.8, 51.7)
- added SW30: SW_SPST, Button_Switch_THT:Tactile_Switch_12x12x7.3_mm, F.Cu at (135.2, 75.8)
- added SW4: Rotary_Encoder_Switch, Rotary_Encoder:RotaryEncoder_Alps_EC12E-Switch_Vertical_H20mm_CircularMountingHoles, F.Cu at (128.9, 51.7)
- added SW5: SW_SPST, Button_Switch_THT:Tactile_Switch_12x12x7.3_mm, F.Cu at (242.8, 62.7)
- added SW6: SW_SPST, Button_Switch_THT:Tactile_Switch_12x12x7.3_mm, F.Cu at (255.4, 62.7)
- added SW7: SW_SPST, Button_Switch_THT:Tactile_Switch_12x12x7.3_mm, F.Cu at (242.8, 78.8)
- added SW8: SW_SPST, Button_Switch_THT:Tactile_Switch_12x12x7.3_mm, F.Cu at (255.4, 78.8)
- added SW9: SW_SPST, Button_Switch_THT:Tactile_Switch_12x12x7.3_mm, F.Cu at (242.8, 94.9)
- added U1: AMS1117-3.3, Package_TO_SOT_SMD:SOT-223-3_TabPin2, F.Cu at (165.4, 27.4)
Other:
- board outline added: 239 x 80 mm

Commit message: Revert "Revert "added a reset button to the power board""
This reverts commit f20825db904c66ff1a5b44b22e19a70ce58abb56.
Parts:
- removed C1: 10uf, Capacitor_Tantalum_SMD:CP_EIA-3216-18_Kemet-A
- removed C2: 22uf, Capacitor_Tantalum_SMD:CP_EIA-3216-18_Kemet-A
- removed D10, D11, D12, D13, D14, D15, D16, D17, D18, D19, D20, D21, D22, D23, D24, D25, D26, D27, D28, D29, D30, D5, D6, D7, D8, D9: D_ALT, Diode_SMD:D_SOD-123
- removed J1: POWER_BOARD, Connector_PinSocket_2.54mm:PinSocket_1x07_P2.54mm_Vertical
- removed J2: AUDIO_BOARD, Connector_PinSocket_2.54mm:PinSocket_1x10_P2.54mm_Vertical
- removed J3: Raspberry_Pi_2_3, Connector_PinHeader_2.54mm:PinHeader_2x20_P2.54mm_Vertical
- removed J4: MICROPHONE, Connector_PinSocket_2.54mm:PinSocket_1x02_P2.54mm_Vertical
- removed REF** (x4): MountingHole_3.2mm_M3, MountingHole:MountingHole_3.2mm_M3
- removed SW1, SW2, SW3, SW4: Rotary_Encoder_Switch, Rotary_Encoder:RotaryEncoder_Alps_EC12E-Switch_Vertical_H20mm_CircularMountingHoles
- removed SW10, SW11, SW12, SW13, SW14, SW15, SW16, SW17, SW18, SW19, SW20, SW21, SW22, SW23, SW24, SW25, SW26, SW27, SW28, SW29, SW30, SW5, SW6, SW7, SW8, SW9: SW_SPST, Button_Switch_THT:Tactile_Switch_12x12x7.3_mm
- removed U1: AMS1117-3.3, Package_TO_SOT_SMD:SOT-223-3_TabPin2
Other:
- board outline removed
