File: OTTO-main/OTTO-main.kicad_pcb (KiCad board)
At the start: 2 copper layers, 41 parts, among them IC1 74HC125, U2 STM32F103CBTx, U3 ILI9341, U4 MCP602, Y1 8mhz

Commit message: progresses in the mainboard wiring
Parts:
- removed C10, C11, C12, C13, C14: 0.1uF, Capacitor_SMD:C_0805_2012Metric
- removed IC1: 74HC125, Package_SO:SOIC-14_3.9x8.7mm_P1.27mm
- removed R10, R11, R12, R3, R4, R5, R6, R7, R8, R9: 10K, Resistor_SMD:R_0805_2012Metric
- removed R13, R15: 1.5K, Resistor_SMD:R_0805_2012Metric
- removed R14: 470K, Resistor_SMD:R_0805_2012Metric
- removed R16: 820K, Resistor_SMD:R_0805_2012Metric
- removed R17, R19: 1K, Resistor_SMD:R_0805_2012Metric
- removed R18: 15K, Resistor_SMD:R_0805_2012Metric
- removed U4: MCP602, Package_SO:SOIC-8_3.9x4.9mm_P1.27mm
- added D10: D_ALT, Diode_SMD:D_SOD-123, B.Cu at (264.6, 54.2)
- added D11: D_ALT, Diode_SMD:D_SOD-123, B.Cu at (249.6, 84.2)
- added D12: D_ALT, Diode_SMD:D_SOD-123, B.Cu at (264.6, 84.2)
- added D13: 1N4148, Diode_SMD:D_SOD-123, B.Cu at (47.1, 55.2)
- added D14: 1N4148, Diode_SMD:D_SOD-123, B.Cu at (77.1, 55.2)
- added D15: D_ALT, Diode_SMD:D_SOD-123, B.Cu at (39.6, 84.2)
- added D16: D_ALT, Diode_SMD:D_SOD-123, B.Cu at (54.6, 84.2)
- added D17: D_ALT, Diode_SMD:D_SOD-123, B.Cu at (69.6, 84.2)
- added D18: D_ALT, Diode_SMD:D_SOD-123, B.Cu at (84.6, 84.2)
- added D19: D_ALT, Diode_SMD:D_SOD-123, B.Cu at (99.6, 84.2)
- added D20: D_ALT, Diode_SMD:D_SOD-123, B.Cu at (114.6, 84.2)
- added D21: D_ALT, Diode_SMD:D_SOD-123, B.Cu at (129.6, 84.2)
- added D22: D_ALT, Diode_SMD:D_SOD-123, B.Cu at (144.6, 84.2)
- added D23: D_ALT, Diode_SMD:D_SOD-123, B.Cu at (249.6, 69.2)
- added D24: D_ALT, Diode_SMD:D_SOD-123, B.Cu at (264.6, 69.2)
- added D25: D_ALT, Diode_SMD:D_SOD-123, B.Cu at (249.6, 99.2)
- added D26: D_ALT, Diode_SMD:D_SOD-123, B.Cu at (264.6, 99.2)
- added D27: 1N4148, Diode_SMD:D_SOD-123, B.Cu at (107.1, 55.2)
- added D28: 1N4148, Diode_SMD:D_SOD-123, B.Cu at (137.1, 55.2)
- added D29: D_ALT, Diode_SMD:D_SOD-123, B.Cu at (39.6, 99.2)
- added D30: D_ALT, Diode_SMD:D_SOD-123, B.Cu at (54.6, 99.2)
- added D31: D_ALT, Diode_SMD:D_SOD-123, B.Cu at (69.6, 99.2)
- added D32: D_ALT, Diode_SMD:D_SOD-123, B.Cu at (84.6, 99.2)
- added D33: D_ALT, Diode_SMD:D_SOD-123, B.Cu at (99.6, 99.2)
- added D34: D_ALT, Diode_SMD:D_SOD-123, B.Cu at (114.6, 99.2)
- added D35: D_ALT, Diode_SMD:D_SOD-123, B.Cu at (129.6, 99.2)
- added D36: D_ALT, Diode_SMD:D_SOD-123, B.Cu at (144.6, 99.2)
- added D37: D_ALT, Diode_SMD:D_SOD-123, B.Cu at (159.6, 99.2)
- added D38: D_ALT, Diode_SMD:D_SOD-123, B.Cu at (174.6, 99.2)
- added D39: D_ALT, Diode_SMD:D_SOD-123, B.Cu at (189.6, 99.2)
- added D40: D_ALT, Diode_SMD:D_SOD-123, B.Cu at (204.6, 99.2)
- added D41: D_ALT, Diode_SMD:D_SOD-123, B.Cu at (219.6, 99.2)
- added D42: D_ALT, Diode_SMD:D_SOD-123, B.Cu at (234.6, 99.2)
- added D43: WS2812B, LED_SMD:WS2812B_3535, F.Cu at (39.6, 72.2)
- added D44: WS2812B, LED_SMD:WS2812B_3535, F.Cu at (54.6, 72.2)
- added D45: WS2812B, LED_SMD:WS2812B_3535, F.Cu at (69.6, 72.2)
- added D46: WS2812B, LED_SMD:WS2812B_3535, F.Cu at (84.6, 72.2)
- added D47: WS2812B, LED_SMD:WS2812B_3535, F.Cu at (99.6, 72.2)
- added D48: WS2812B, LED_SMD:WS2812B_3535, F.Cu at (114.6, 72.2)
- added D49: WS2812B, LED_SMD:WS2812B_3535, F.Cu at (129.6, 72.2)
- added D5: D_ALT, Diode_SMD:D_SOD-123, B.Cu at (99.6, 69.2)
- added D50: WS2812B, LED_SMD:WS2812B_3535, F.Cu at (144.6, 72.2)
- added D51: WS2812B, LED_SMD:WS2812B_3535, F.Cu at (39.6, 87.2)
- added D52: WS2812B, LED_SMD:WS2812B_3535, F.Cu at (54.6, 87.2)
- added D53: WS2812B, LED_SMD:WS2812B_3535, F.Cu at (69.6, 87.2)
- added D54: WS2812B, LED_SMD:WS2812B_3535, F.Cu at (84.6, 87.2)
- added D55: WS2812B, LED_SMD:WS2812B_3535, F.Cu at (99.6, 87.2)
- added D56: WS2812B, LED_SMD:WS2812B_3535, F.Cu at (114.6, 87.2)
- added D57: WS2812B, LED_SMD:WS2812B_3535, F.Cu at (129.6, 87.2)
- added D58: WS2812B, LED_SMD:WS2812B_3535, F.Cu at (144.6, 87.2)
- added D59: WS2812B, LED_SMD:WS2812B_3535, F.Cu at (39.6, 102.2)
- added D6: D_ALT, Diode_SMD:D_SOD-123, B.Cu at (114.6, 69.2)
- added D60: WS2812B, LED_SMD:WS2812B_3535, F.Cu at (54.6, 102.2)
- added D61: WS2812B, LED_SMD:WS2812B_3535, F.Cu at (69.6, 102.2)
- added D62: WS2812B, LED_SMD:WS2812B_3535, F.Cu at (84.6, 102.2)
- added D63: WS2812B, LED_SMD:WS2812B_3535, F.Cu at (99.6, 102.2)
- added D64: WS2812B, LED_SMD:WS2812B_3535, F.Cu at (114.6, 102.2)
- added D65: WS2812B, LED_SMD:WS2812B_3535, F.Cu at (129.6, 102.2)
- added D66: WS2812B, LED_SMD:WS2812B_3535, F.Cu at (144.6, 102.2)
- added D67: WS2812B, LED_SMD:WS2812B_3535, F.Cu at (159.6, 102.2)
- added D68: WS2812B, LED_SMD:WS2812B_3535, F.Cu at (174.6, 102.2)
- added D69: WS2812B, LED_SMD:WS2812B_3535, F.Cu at (189.6, 102.2)
- added D7: D_ALT, Diode_SMD:D_SOD-123, B.Cu at (129.6, 69.2)
- added D70: WS2812B, LED_SMD:WS2812B_3535, F.Cu at (204.6, 102.2)
- added D71: WS2812B, LED_SMD:WS2812B_3535, F.Cu at (219.6, 102.2)
- added D72: WS2812B, LED_SMD:WS2812B_3535, F.Cu at (234.6, 102.2)
- added D73: WS2812B, LED_SMD:WS2812B_3535, F.Cu at (249.6, 102.2)
- added D74: WS2812B, LED_SMD:WS2812B_3535, F.Cu at (264.6, 102.2)
- added D75: WS2812B, LED_SMD:WS2812B_3535, F.Cu at (249.6, 87.2)
- added D76: WS2812B, LED_SMD:WS2812B_3535, F.Cu at (264.6, 87.2)
- added D77: WS2812B, LED_SMD:WS2812B_3535, F.Cu at (249.6, 72.2)
- added D78: WS2812B, LED_SMD:WS2812B_3535, F.Cu at (264.6, 72.2)
- added D79: WS2812B, LED_SMD:WS2812B_3535, F.Cu at (249.6, 57.2)
- added D8: D_ALT, Diode_SMD:D_SOD-123, B.Cu at (144.6, 69.2)
- added D80: WS2812B, LED_SMD:WS2812B_3535, F.Cu at (264.6, 57.2)
- added D9: D_ALT, Diode_SMD:D_SOD-123, B.Cu at (249.6, 54.2)
- added J1: POWER_BOARD, Connector_PinSocket_2.54mm:PinSocket_1x10_P2.54mm_Vertical, B.Cu at (163.3, 41.2)
- added J2: AUDIO_BOARD, Connector_PinSocket_2.54mm:PinSocket_1x10_P2.54mm_Vertical, B.Cu at (239.3, 67.3)
- added J3: Raspberry_Pi_2_3, Connector_PinHeader_2.54mm:PinHeader_2x20_P2.54mm_Vertical, F.Cu at (105.2, 112.1)
- added J4: MICROPHONE, Connector_PinSocket_2.54mm:PinSocket_1x02_P2.54mm_Vertical, B.Cu at (271.8, 109.3)
- added J5: Conn_01x24, Connector_FFC-FPC:JUSHUO_AFC07-S24FCC-00, F.Cu at (260.6, 115.2)
- added R20: 3.9, Resistor_SMD:R_0805_2012Metric, F.Cu at (220.1, 44.1)
- added SW1: SW_SPST, Button_Switch_SMD:SILICONE_BUTTON_10MM_4X4WIDE, F.Cu at (39.6, 72.2)
- added SW10: SW_SPST, Button_Switch_SMD:SILICONE_BUTTON_10MM_4X4WIDE, F.Cu at (264.6, 57.2)
- added SW11: SW_SPST, Button_Switch_SMD:SILICONE_BUTTON_10MM_4X4WIDE, F.Cu at (249.6, 87.2)
- added SW12: SW_SPST, Button_Switch_SMD:SILICONE_BUTTON_10MM_4X4WIDE, F.Cu at (264.6, 87.2)
- added SW13: Rotary_Encoder_Switch, Rotary_Encoder:PEC11S-929K-S0015, F.Cu at (47.1, 52.2)
- added SW14: Rotary_Encoder_Switch, Rotary_Encoder:PEC11S-929K-S0015, F.Cu at (77.1, 52.2)
- added SW15: SW_SPST, Button_Switch_SMD:SILICONE_BUTTON_10MM_4X4WIDE, F.Cu at (39.6, 87.2)
- added SW16: SW_SPST, Button_Switch_SMD:SILICONE_BUTTON_10MM_4X4WIDE, F.Cu at (54.6, 87.2)
- added SW17: SW_SPST, Button_Switch_SMD:SILICONE_BUTTON_10MM_4X4WIDE, F.Cu at (69.6, 87.2)
- added SW18: SW_SPST, Button_Switch_SMD:SILICONE_BUTTON_10MM_4X4WIDE, F.Cu at (84.6, 87.2)
- added SW19: SW_SPST, Button_Switch_SMD:SILICONE_BUTTON_10MM_4X4WIDE, F.Cu at (99.6, 87.2)
- added SW2: SW_SPST, Button_Switch_SMD:SILICONE_BUTTON_10MM_4X4WIDE, F.Cu at (54.6, 72.2)
- added SW20: SW_SPST, Button_Switch_SMD:SILICONE_BUTTON_10MM_4X4WIDE, F.Cu at (114.6, 87.2)
- added SW21: SW_SPST, Button_Switch_SMD:SILICONE_BUTTON_10MM_4X4WIDE, F.Cu at (129.6, 87.2)
- added SW22: SW_SPST, Button_Switch_SMD:SILICONE_BUTTON_10MM_4X4WIDE, F.Cu at (144.6, 87.2)
- added SW23: SW_SPST, Button_Switch_SMD:SILICONE_BUTTON_10MM_4X4WIDE, F.Cu at (249.6, 72.2)
- added SW24: SW_SPST, Button_Switch_SMD:SILICONE_BUTTON_10MM_4X4WIDE, F.Cu at (264.6, 72.2)
- added SW25: SW_SPST, Button_Switch_SMD:SILICONE_BUTTON_10MM_4X4WIDE, F.Cu at (249.6, 102.2)
- added SW26: SW_SPST, Button_Switch_SMD:SILICONE_BUTTON_10MM_4X4WIDE, F.Cu at (264.6, 102.2)
- added SW27: Rotary_Encoder_Switch, Rotary_Encoder:PEC11S-929K-S0015, F.Cu at (107.1, 52.2)
- added SW28: Rotary_Encoder_Switch, Rotary_Encoder:PEC11S-929K-S0015, F.Cu at (137.1, 52.2)
- added SW29: SW_SPST, Button_Switch_SMD:SILICONE_BUTTON_10MM_4X4WIDE, F.Cu at (39.6, 102.2)
- added SW3: SW_SPST, Button_Switch_SMD:SILICONE_BUTTON_10MM_4X4WIDE, F.Cu at (69.6, 72.2)
- added SW30: SW_SPST, Button_Switch_SMD:SILICONE_BUTTON_10MM_4X4WIDE, F.Cu at (54.6, 102.2)
- added SW31: SW_SPST, Button_Switch_SMD:SILICONE_BUTTON_10MM_4X4WIDE, F.Cu at (69.6, 102.2)
- added SW32: SW_SPST, Button_Switch_SMD:SILICONE_BUTTON_10MM_4X4WIDE, F.Cu at (84.6, 102.2)
- added SW33: SW_SPST, Button_Switch_SMD:SILICONE_BUTTON_10MM_4X4WIDE, F.Cu at (99.6, 102.2)
- added SW34: SW_SPST, Button_Switch_SMD:SILICONE_BUTTON_10MM_4X4WIDE, F.Cu at (114.6, 102.2)
- added SW35: SW_SPST, Button_Switch_SMD:SILICONE_BUTTON_10MM_4X4WIDE, F.Cu at (129.6, 102.2)
- added SW36: SW_SPST, Button_Switch_SMD:SILICONE_BUTTON_10MM_4X4WIDE, F.Cu at (144.6, 102.2)
- added SW37: SW_SPST, Button_Switch_SMD:SILICONE_BUTTON_10MM_4X4WIDE, F.Cu at (159.6, 102.2)
- added SW38: SW_SPST, Button_Switch_SMD:SILICONE_BUTTON_10MM_4X4WIDE, F.Cu at (174.6, 102.2)
- added SW39: SW_SPST, Button_Switch_SMD:SILICONE_BUTTON_10MM_4X4WIDE, F.Cu at (189.6, 102.2)
- added SW4: SW_SPST, Button_Switch_SMD:SILICONE_BUTTON_10MM_4X4WIDE, F.Cu at (84.6, 72.2)
- added SW40: SW_SPST, Button_Switch_SMD:SILICONE_BUTTON_10MM_4X4WIDE, F.Cu at (204.6, 102.2)
- added SW41: SW_SPST, Button_Switch_SMD:SILICONE_BUTTON_10MM_4X4WIDE, F.Cu at (219.6, 102.2)
- added SW42: SW_SPST, Button_Switch_SMD:SILICONE_BUTTON_10MM_4X4WIDE, F.Cu at (234.6, 102.2)
- added SW5: SW_SPST, Button_Switch_SMD:SILICONE_BUTTON_10MM_4X4WIDE, F.Cu at (99.6, 72.2)
- added SW6: SW_SPST, Button_Switch_SMD:SILICONE_BUTTON_10MM_4X4WIDE, F.Cu at (114.6, 72.2)
- added SW7: SW_SPST, Button_Switch_SMD:SILICONE_BUTTON_10MM_4X4WIDE, F.Cu at (129.6, 72.2)
- added SW8: SW_SPST, Button_Switch_SMD:SILICONE_BUTTON_10MM_4X4WIDE, F.Cu at (144.6, 72.2)
- added SW9: SW_SPST, Button_Switch_SMD:SILICONE_BUTTON_10MM_4X4WIDE, F.Cu at (249.6, 57.2)
- added U1: STM32F103RETx, Package_QFP:LQFP-64_10x10mm_P0.5mm, F.Cu at (161.1, 77.6)
- D1, D2, D3, D4: value 1N4148 -> D_ALT; footprint Diode_SMD:D_SOD-123v -> Diode_SMD:D_SOD-123; moved to B.Cu
- U2: value STM32F103CBTx -> 74AHCT1G125; footprint Package_QFP:LQFP-48_7x7mm_P0.5mm -> Package_TO_SOT_SMD:SOT-23-5; moved to B.Cu
- U3: footprint Connector_PinHeader_2.54mm:PinHeader_1x18_P2.54mm_Horizontal -> Display:ILI_DISPLAY
- moved U3 282.6 mm to (197.1, 70.6), turned to 180 degrees
- moved C4 245.2 mm to (165.9, 68.7)
- moved C5 238.5 mm to (164.8, 87.3), turned to 270 degrees
- moved Y1 226.9 mm to (164.6, 64.6), turned to 180 degrees
- moved C3 226.1 mm to (152.3, 83.8), turned to 270 degrees
- moved C8 225.7 mm to (166.1, 59.7), turned to 90 degrees
- moved C9 221.6 mm to (163.0, 59.7), turned to 90 degrees
- moved L1 213.7 mm to (158.6, 55.9), turned to 180 degrees
- moved C6 208.3 mm to (158.6, 61.9), turned to 180 degrees
- moved C7 207.4 mm to (158.6, 58.9), turned to 180 degrees
- moved R2 195.6 mm to (117.3, 114.5), turned to 90 degrees
- moved R1 187.4 mm to (114.5, 114.5), turned to 270 degrees
- moved D3 133.3 mm to (69.6, 69.2), turned to 180 degrees
- moved U2 128.8 mm to (34.6, 65.6), turned to 90 degrees
- moved D4 117.4 mm to (84.6, 69.2), turned to 180 degrees
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Connections:
- net +5V renamed Net-(J3-Pad1)
- C3 pad 1: +3V3 -> 3V3
- C3 pad 2: GNDREF -> GND
- C4 pad 1: +3V3 -> 3V3
- C4 pad 2: GNDREF -> GND
- C5 pad 1: +3V3 -> 3V3
- C5 pad 2: GNDREF -> GND
- C6 pad 2: GNDREF -> GND
- C7 pad 2: GNDREF -> GND
- C8 pad 2: GNDREF -> GND
- C9 pad 2: GNDREF -> GND
- L1 pad 2: +3V3 -> 3V3
- R1 pad 1: SCL -> SDA
- U2 pad 1: Net-(U2-Pad1) -> GND
- U2 pad 3: Net-(U2-Pad3) -> GND
- U2 pad 4: Net-(U2-Pad4) -> LEDIN
- U2 pad 5: OSC_IN -> 5V
- U3 pad 1: GNDREF -> GND
- U3 pad 11: GNDREF -> GND
- U3 pad 12: GNDREF -> GND
- U3 pad 13: GNDREF -> GND
- U3 pad 14: GNDREF -> GND
- U3 pad 15: Net-(U3-Pad15) -> (no net)
- U3 pad 16: Net-(U3-Pad16) -> (no net)
- U3 pad 17: Net-(U3-Pad17) -> (no net)
- U3 pad 18: Net-(U3-Pad18) -> (no net)
- U3 pad 8: GNDREF -> GND
- U3 pad 9: Net-(U3-Pad9) -> 3V3
Routing:
- net ROW2: track 0.00 -> 427.9 mm, vias 0 -> 8
- net 5V: track 0.00 -> 417.7 mm, vias 0 -> 81
- net ROW1: track 0.00 -> 413.6 mm, vias 0 -> 8
- net COL1: track 0.00 -> 393.2 mm, vias 0 -> 4
- net COL2: track 0.00 -> 361.3 mm, vias 0 -> 4
- net COL3: track 0.00 -> 330.0 mm, vias 0 -> 4
- net ROW3: track 0.00 -> 307.1 mm, vias 0 -> 2
- net COL4: track 0.00 -> 299.2 mm, vias 0 -> 4
- net COL9: track 0.00 -> 281.7 mm, vias 0 -> 8
- net COL10: track 0.00 -> 276.3 mm, vias 0 -> 6
- net SENSE_PIN: track 0.00 -> 272.3 mm
- net COL13: track 0.00 -> 270.3 mm, vias 0 -> 7
- net COL5: track 0.00 -> 268.4 mm, vias 0 -> 4
- net OUT_PIN: track 0.00 -> 264.2 mm, vias 0 -> 1
- net DOK_OUT: track 0.00 -> 244.8 mm, vias 0 -> 3
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- added copper zone on F.Cu, net 3V3
- added copper zone on F.Cu, net 5V
- added copper zone on B.Cu, net GND
Other:
- board outline added: 247 x 81 mm
- copper layers 2 -> 4
- net class 5V added: clearance 0.2, trace_width 0.6, via_dia 1, via_drill 0.5
