File: OTTO-main/OTTO-main.sch (KiCad schematic (older format))
At the start: 109 parts, among them IC1 74HC125, J1 POWER_BOARD, J2 AUDIO_BOARD, J3 Raspberry_Pi_2_3, J4 MICROPHONE, SW1 Rotary_Encoder_Switch, SW10 SW_SPST, SW11 SW_SPST, SW12 SW_SPST, SW13 SW_SPST, SW14 SW_SPST, SW15 SW_SPST, SW16 SW_SPST, SW17 SW_SPST, SW18 SW_SPST, SW19 SW_SPST, SW2 Rotary_Encoder_Switch, SW20 SW_SPST, SW21 SW_SPST, SW22 SW_SPST, SW23 SW_SPST, SW24 SW_SPST, SW25 SW_SPST, SW26 SW_SPST, SW27 SW_SPST, SW28 SW_SPST, SW29 SW_SPST, SW3 Rotary_Encoder_Switch, SW30 SW_SPST, SW4 Rotary_Encoder_Switch, SW5 SW_SPST, SW6 SW_SPST, SW7 SW_SPST, SW8 SW_SPST, SW9 SW_SPST, U2 STM32F103CBTx, U3 ILI9341, U4 MCP602, Y1 8mhz

Commit message: Revert "added a reset button to the power board"
This reverts commit bbfaa2fb8df27d7f63d1a584e9f51fc8f5fa6fe3.
Parts:
- removed D31, D32, D33, D34, D35, D36: WS2812B, LED_SMD:WS2812B_3535, symbol LED:WS2812B
- SW10, SW11, SW12, SW13, SW14, SW15, SW16, SW17, SW18, SW19, SW20, SW21, SW22, SW23, SW24, SW25, SW26, SW27, SW28, SW29, SW30, SW5, SW6, SW7, SW8, SW9: footprint Button_Switch_SMD:SILICONE_BUTTON_10MM_4X4WIDE -> Button_Switch_THT:Tactile_Switch_12x12x7.3_mm
- renumbered R20 to R?
Connections:
- wire segments 482 -> 464

Commit message: Revert "Revert "added a reset button to the power board""
This reverts commit f20825db904c66ff1a5b44b22e19a70ce58abb56.
Parts:
- added D31, D32, D33, D34, D35, D36: WS2812B, LED_SMD:WS2812B_3535, symbol LED:WS2812B
- SW10, SW11, SW12, SW13, SW14, SW15, SW16, SW17, SW18, SW19, SW20, SW21, SW22, SW23, SW24, SW25, SW26, SW27, SW28, SW29, SW30, SW5, SW6, SW7, SW8, SW9: footprint Button_Switch_THT:Tactile_Switch_12x12x7.3_mm -> Button_Switch_SMD:SILICONE_BUTTON_10MM_4X4WIDE
- gave numbers to parts that had none: 1
Connections:
- wire segments 464 -> 482

Commit message: progresses in the mainboard wiring
Parts:
- removed C10, C11, C12, C13, C14: 0.1uF, Capacitor_SMD:C_0805_2012Metric, symbol Device:C_Small
- removed D10, D11, D12, D13, D14, D15, D16, D17, D18, D19, D20, D21, D22, D23, D24, D25, D26, D27, D28, D29, D30, D5, D6, D7, D8, D9: D_ALT, Diode_SMD:D_SOD-123, symbol Device:D_ALT
- removed D31, D32, D33, D34, D35, D36: WS2812B, LED_SMD:WS2812B_3535, symbol LED:WS2812B
- removed IC1: 74HC125, Package_SO:SOIC-14_3.9x8.7mm_P1.27mm, symbol 74HC125N:74HC125N
- removed J1: POWER_BOARD, Connector_PinSocket_2.54mm:PinSocket_1x07_P2.54mm_Vertical, symbol Connector_Generic:Conn_01x07
- removed R10, R11, R12, R3, R4, R5, R6, R7, R8, R9: 10K, Resistor_SMD:R_0805_2012Metric, symbol Device:R_US
- removed R13, R15: 1.5K, Resistor_SMD:R_0805_2012Metric, symbol Device:R_US
- removed R14: 470K, Resistor_SMD:R_0805_2012Metric, symbol Device:R_US
- removed R16: 820K, Resistor_SMD:R_0805_2012Metric, symbol Device:R_US
- removed R17, R19: 1K, Resistor_SMD:R_0805_2012Metric, symbol Device:R_US
- removed R18: 15K, Resistor_SMD:R_0805_2012Metric, symbol Device:R_US
- removed SW10, SW11, SW12, SW13, SW14, SW15, SW16, SW17, SW18, SW19, SW20, SW21, SW22, SW23, SW24, SW25, SW26, SW27, SW28, SW29, SW30, SW5, SW6, SW7, SW8, SW9: SW_SPST, Button_Switch_SMD:SILICONE_BUTTON_10MM_4X4WIDE, symbol Switch:SW_SPST
- removed U2: STM32F103CBTx, Package_QFP:LQFP-48_7x7mm_P0.5mm, symbol MCU_ST_STM32F1:STM32F103CBTx
- removed U4: MCP602, Package_SO:SOIC-8_3.9x4.9mm_P1.27mm, symbol Amplifier_Operational:MCP602
- added J1: POWER_BOARD, Connector_PinSocket_2.54mm:PinSocket_1x10_P2.54mm_Vertical, symbol Connector_Generic:Conn_01x10
- added J5: Conn_01x24, Connector_FFC-FPC:JUSHUO_AFC07-S24FCC-00, symbol Connector_Generic:Conn_01x24
- added U1: STM32F103RETx, Package_QFP:LQFP-64_10x10mm_P0.5mm, symbol MCU_ST_STM32F1:STM32F103RETx
- D13: renamed from D1; footprint Diode_SMD:D_SOD-123v -> Diode_SMD:D_SOD-123
- D14: renamed from D2; footprint Diode_SMD:D_SOD-123v -> Diode_SMD:D_SOD-123
- D27: renamed from D3; footprint Diode_SMD:D_SOD-123v -> Diode_SMD:D_SOD-123
- D28: renamed from D4; footprint Diode_SMD:D_SOD-123v -> Diode_SMD:D_SOD-123
- SW13: renamed from SW1; footprint Rotary_Encoder:RotaryEncoder_Alps_EC12E-Switch_Vertical_H20mm_CircularMountingHoles -> Rotary_Encoder:PEC11S-929K-S0015
- SW14: renamed from SW2; footprint Rotary_Encoder:RotaryEncoder_Alps_EC12E-Switch_Vertical_H20mm_CircularMountingHoles -> Rotary_Encoder:PEC11S-929K-S0015
- SW27: renamed from SW3; footprint Rotary_Encoder:RotaryEncoder_Alps_EC12E-Switch_Vertical_H20mm_CircularMountingHoles -> Rotary_Encoder:PEC11S-929K-S0015
- SW28: renamed from SW4; footprint Rotary_Encoder:RotaryEncoder_Alps_EC12E-Switch_Vertical_H20mm_CircularMountingHoles -> Rotary_Encoder:PEC11S-929K-S0015
- U3: footprint Connector_PinHeader_2.54mm:PinHeader_1x18_P2.54mm_Horizontal -> Display:ILI_DISPLAY
Connections:
- net labels added: CHG_OUT, COL14, DOK_OUT, ENC1_A, ENC1_B, ENC2_A, ENC2_B, ENC3_A, ENC3_B, ENC4_A, ENC4_B, KBLED, LEDIN, ROW6, ROW7
- net labels removed: A_PIN, D_PIN, INT_PIN, LED_POW, WS2812
- wire segments 482 -> 225
- no-connect marks 5 -> 32

Commit message: re-wired the stm32 to optimize the routing
Connections:
- no-connect marks 32 -> 18
Changed lines of the file:
@@
 	15700 10500 17400 10500
+Wire Wire Line
+	16550 9350 16200 9350
+Text GLabel 16200 9350 0    50   Input ~ 0
+ROW4
+Wire Wire Line
+	16550 9450 16200 9450
+Text GLabel 16200 9450 0    50   Input ~ 0
+ROW5
 Wire Wire Line
 	16550 7950 16200 7950
 Text GLabel 16200 7950 0    50   Input ~ 0
-ROW4
+COL1
 Wire Wire Line
 	16550 8050 16200 8050
 Text GLabel 16200 8050 0    50   Input ~ 0
-ROW5
+COL2
 Wire Wire Line
 	16550 8150 16200 8150
 Text GLabel 16200 8150 0    50   Input ~ 0
-COL1
+COL3
 Wire Wire Line
 	16550 8250 16200 8250
 Text GLabel 16200 8250 0    50   Input ~ 0
-COL2
+COL4
 Wire Wire Line
 	16550 8350 16200 8350
 Text GLabel 16200 8350 0    50   Input ~ 0
-COL3
+COL5
 Wire Wire Line
 	16550 8450 16200 8450
 Text GLabel 16200 8450 0    50   Input ~ 0
-COL4
+COL6
 Wire Wire Line
 	16550 8550 16200 8550
 Text GLabel 16200 8550 0    50   Input ~ 0
-COL5
+COL7
 Wire Wire Line
 	16550 8650 16200 8650
 Text GLabel 16200 8650 0    50   Input ~ 0
-COL6
+COL8
 Wire Wire Line
 	16550 8750 16200 8750
 Text GLabel 16200 8750 0    50   Input ~ 0
-COL7
+COL9
 Wire Wire Line
 	16550 8850 16200 8850
 Text GLabel 16200 8850 0    50   Input ~ 0
-COL8
+COL10
 Wire Wire Line
 	16550 8950 16200 8950
 Text GLabel 16200 8950 0    50   Input ~ 0
-COL9
+COL11
 Wire Wire Line
 	16550 9050 16200 9050
 Text GLabel 16200 9050 0    50   Input ~ 0
-COL10
+COL12
 Wire Wire Line
 	16550 9150 16200 9150
 Text GLabel 16200 9150 0    50   Input ~ 0
-COL11
-Wire Wire Line
-	16550 9250 16200 9250
-Text GLabel 16200 9250 0    50   Input ~ 0
-COL12
-Wire Wire Line
-	16550 9350 16200 9350
-Text GLabel 16200 9350 0    50   Input ~ 0
 COL13
 Wire Wire Line
@@
 Wire Wire Line
 	16250 6100 16550 6100
-$Comp
-L MCU_ST_STM32F1:STM32F103RETx U1
-U 1 1 5BB77EF9
-P 2150 3450
-F 0 "U1" H 2150 3400 50  0000 C CNN
-F 1 "STM32F103RETx" H 2150 3550 50  0000 C CNN
-F 2 "Package_QFP:LQFP-64_10x10mm_P0.5mm" H 1550 1750 50  0001 R CNN
-F 3 "http://www.st.com/st-web-ui/static/active/en/resource/technical/document/datasheet/CD00191185.pdf" H 2150 3450 50  0001 C CNN
-	1    2150 3450
-	1    0    0    -1
-$EndComp
 Wire Wire Line
 	2250 1550 2350 1550
@@
 $EndSheet
 Wire Wire Line
-	16550 9450 16200 9450
-Text GLabel 16200 9450 0    50   Input ~ 0
+	16550 9250 16200 9250
+Text GLabel 16200 9250 0    50   Input ~ 0
 COL14
 Wire Wire Line
-	2850 2350 3350 2350
-Text GLabel 3350 2350 2    50   Input ~ 0
+	2850 4450 3350 4450
+Text GLabel 3350 4450 2    50   Input ~ 0
 COL10
 Wire Wire Line
-	2850 2450 3350 2450
-Text GLabel 3350 2450 2    50   Input ~ 0
+	1450 4850 950  4850
+Text GLabel 950  4850 0    50   Input ~ 0
 COL11
 Wire Wire Line
-	2850 2550 3350 2550
-Text GLabel 3350 2550 2    50   Input ~ 0
+	1450 4950 950  4950
+Text GLabel 950  4950 0    50   Input ~ 0
 COL12
 Wire Wire Line
-	1450 3950 950  3950
-Text GLabel 950  3950 0    50   Input ~ 0
+	1450 5050 950  5050
+Text GLabel 950  5050 0    50   Input ~ 0
 COL13
-Wire Wire Line
-	1450 4050 950  4050
-Text GLabel 950  4050 0    50   Input ~ 0
-COL14
-Text GLabel 3350 3550 2    50   Input ~ 0
-ROW1
-Wire Wire Line
-	2850 3550 3350 3550
-Text GLabel 3350 4550 2    50   Input ~ 0
-ROW3
-Wire Wire Line
-	2850 4550 3350 4550
-Text GLabel 3350 3650 2    50   Input ~ 0
-ROW2
-Wire Wire Line
-	2850 3650 3350 3650
 Wire Wire Line
 	1450 3550 950  3550
 Text GLabel 950  3550 0    50   Input ~ 0
-COL1
-Wire Wire Line
-	1450 3650 950  3650
-Text GLabel 950  3650 0    50   Input ~ 0
-COL2
-Wire Wire Line
-	1450 3750 950  3750
-Text GLabel 950  3750 0    50   Input ~ 0
-COL3
-Wire Wire Line
-	1450 3850 950  3850
-Text GLabel 950  3850 0    50   Input ~ 0
-COL4
-Wire Wire Line
-	2850 1850 3350 1850
-Text GLabel 3350 1850 2    50   Input ~ 0
-COL5
-Wire Wire Line
-	2850 1950 3350 1950
-Text GLabel 3350 1950 2    50   Input ~ 0
-COL6
-Wire Wire Line
-	2850 2050 3350 2050
-Text GLabel 3350 2050 2    50   Input ~ 0
-COL7
-Wire Wire Line
-	2850 2150 3350 2150
-Text GLabel 3350 2150 2    50   Input ~ 0
-COL8
-Wire Wire Line
-	2850 2250 3350 2250
-Text GLabel 3350 2250 2    50   Input ~ 0
-COL9
+COL14
+Text GLabel 3350 2950 2    50   Input ~ 0
+ROW1
+Wire Wire Line
+	2850 2950 3350 2950
+Text GLabel 3350 3150 2    50   Input ~ 0
+ROW3
+Wire Wire Line
+	2850 3150 3350 3150
+Text GLabel 3350 3050 2    50   Input ~ 0
+ROW2
+Wire Wire Line
+	2850 3050 3350 3050
 Wire Wire Line
 	2850 3250 3350 3250
 Text GLabel 3350 3250 2    50   Input ~ 0
-ROW4
+COL1
 Wire Wire Line
 	2850 3350 3350 3350
 Text GLabel 3350 3350 2    50   Input ~ 0
+COL2
+Wire Wire Line
+	1450 4550 950  4550
+Text GLabel 950  4550 0    50   Input ~ 0
+COL3
+Wire Wire Line
+	1450 4650 950  4650
+Text GLabel 950  4650 0    50   Input ~ 0
+COL4
+Wire Wire Line
+	1450 4750 950  4750
+Text GLabel 950  4750 0    50   Input ~ 0
+COL5
+Wire Wire Line
+	2850 3850 3350 3850
+Text GLabel 3350 3850 2    50   Input ~ 0
+COL6
+Wire Wire Line
+	2850 3950 3350 3950
+Text GLabel 3350 3950 2    50   Input ~ 0
+COL7
+Wire Wire Line
+	2850 4050 3350 4050
+Text GLabel 3350 4050 2    50   Input ~ 0
+COL8
+Wire Wire Line
+	2850 4350 3350 4350
+Text GLabel 3350 4350 2    50   Input ~ 0
+COL9
+Wire Wire Line
+	4200 4050 4700 4050
+Text GLabel 4700 4050 2    50   Input ~ 0
+ROW4
+Wire Wire Line
+	4200 4150 4700 4150
+Text GLabel 4700 4150 2    50   Input ~ 0
 ROW5
 Wire Wire Line
@@
 Text GLabel 3350 7850 3    50   Input ~ 0
 ENC4_B
+Text GLabel 3350 4750 2    50   Input ~ 0
+ENC1_B
 Text GLabel 3350 4850 2    50   Input ~ 0
+ENC1_A
+Wire Wire Line
+	2850 4750 3350 4750
+Wire Wire Line
+	2850 4850 3350 4850
+Text GLabel 3350 4950 2    50   Input ~ 0
+ENC2_B
+Wire Wire Line
+	2850 4950 3350 4950
+Text GLabel 950  4450 0    50   Input ~ 0
 ENC4_A
-Text GLabel 3350 4950 2    50   Input ~ 0
-ENC4_B
-Wire Wire Line
-	2850 4850 3350 4850
-Wire Wire Line
-	2850 4950 3350 4950
-Text GLabel 3350 5050 2    50   Input ~ 0
-ENC3_A
-Wire Wire Line
-	2850 5050 3350 5050
-Text GLabel 3350 2650 2    50   Input ~ 0
-ENC1_B
-Wire Wire Line
-	2850 2650 3350 2650
-Text GLabel 3100 2950 2    50   Input ~ 0
+Wire Wire Line
+	1450 4450 950  4450
+Text GLabel 3100 2650 2    50   Input ~ 0
 LEDIN
 Wire Wire Line
-	3100 2950 2850 2950
+	3100 2650 2850 2650
 Text GLabel 16300 1000 0    50   Input ~ 0
 3V3
@@
 	16500 10850 17050 10850
 Wire Wire Line
-	950  4450 1450 4450
-Text GLabel 950  4450 0    50   Input ~ 0
-ENC1_A
-Wire Wire Line
 	950  4350 1450 4350
+Text GLabel 950  4350 0    50   Input ~ 0
+ENC4_B
 Wire Wire Line
 	950  4250 1450 4250
-Text GLabel 950  4350 0    50   Input ~ 0
-ENC2_B
+Wire Wire Line
+	950  4150 1450 4150
 Text GLabel 950  4250 0    50   Input ~ 0
-ENC2_A
-Wire Wire Line
-	950  4150 1450 4150
+ENC3_A
 Text GLabel 950  4150 0    50   Input ~ 0
 ENC3_B
+Wire Wire Line
+	3350 5050 2850 5050
+Text GLabel 3350 5050 2    50   Input ~ 0
+ENC2_A
 NoConn ~ 8900 4500
 NoConn ~ 8900 3300
@@
 NoConn ~ 9600 2500
 NoConn ~ 10500 4600
-NoConn ~ 2850 3050
-NoConn ~ 2850 3150
-NoConn ~ 2850 3850
-NoConn ~ 2850 3950
-NoConn ~ 2850 4050
-NoConn ~ 2850 4450
-NoConn ~ 2850 4350
-NoConn ~ 1450 5050
-NoConn ~ 1450 4950
-NoConn ~ 1450 4850
-NoConn ~ 1450 4750
-NoConn ~ 1450 4650
-NoConn ~ 1450 4550
 NoConn ~ 1450 3350
 Wire Wire Line
@@
 Wire Wire Line
 	16200 9950 16550 9950
-NoConn ~ 2850 4750
 NoConn ~ 2850 4650
 Wire Wire Line
@@
 	10900 3200 11200 3200
 Connection ~ 10900 3200
+$Comp
+L MCU_ST_STM32F1:STM32F103RETx U1
+U 1 1 5BB77EF9
+P 2150 3450
+F 0 "U1" H 2150 3400 50  0000 C CNN
+F 1 "STM32F103RETx" H 2150 3550 50  0000 C CNN
+F 2 "Package_QFP:LQFP-64_10x10mm_P0.5mm" H 1550 1750 50  0001 R CNN
+F 3 "http://www.st.com/st-web-ui/static/active/en/resource/technical/document/datasheet/CD00191185.pdf" H 2150 3450 50  0001 C CNN
+	1    2150 3450
+	1    0    0    -1
+$EndComp
 $EndSCHEMATC

Commit message: added the OTTO-keys files
Changed lines of the file:
@@
 COL9
 Wire Wire Line
-	4200 4050 4700 4050
-Text GLabel 4700 4050 2    50   Input ~ 0
+	1450 3650 950  3650
+Text GLabel 950  3650 0    50   Input ~ 0
 ROW4
 Wire Wire Line
-	4200 4150 4700 4150
-Text GLabel 4700 4150 2    50   Input ~ 0
+	1450 3750 950  3750
+Text GLabel 950  3750 0    50   Input ~ 0
 ROW5
 Wire Wire Line
@@
 	1    0    0    -1
 $EndComp
-Text GLabel 16500 11050 0    50   Input ~ 0
+Text GLabel 16500 11000 0    50   Input ~ 0
 GND
-Text GLabel 16500 10850 0    50   Input ~ 0
+Text GLabel 16500 10800 0    50   Input ~ 0
 5V
-Text GLabel 16500 10950 0    50   Input ~ 0
+Text GLabel 16500 10900 0    50   Input ~ 0
 3V3
 $Comp
 L power:GNDREF #PWR0102
 U 1 1 5BB96502
-P 17050 11050
+P 17050 11000
 AR Path="/5BB96502" Ref="#PWR0102"  Part="1"
 AR Path="/5DEA5FAF/5BB96502" Ref="#PWR?"  Part="1"
-F 0 "#PWR0102" H 17050 10800 50  0001 C CNN
-F 1 "GNDREF" H 17055 10877 50  0000 C CNN
-F 2 "" H 17050 11050 50  0001 C CNN
-F 3 "" H 17050 11050 50  0001 C CNN
-	1    17050 11050
+F 0 "#PWR0102" H 17050 10750 50  0001 C CNN
+F 1 "GNDREF" H 17055 10827 50  0000 C CNN
+F 2 "" H 17050 11000 50  0001 C CNN
+F 3 "" H 17050 11000 50  0001 C CNN
+	1    17050 11000
 	1    0    0    -1
 $EndComp
 Wire Wire Line
-	16500 11050 17050 11050
+	16500 11000 17050 11000
 $Comp
 L power:+3V3 #PWR0103
 U 1 1 5BBA60A9
-P 17050 10950
-F 0 "#PWR0103" H 17050 10800 50  0001 C CNN
-F 1 "+3V3" V 17065 11123 50  0000 C CNN
-F 2 "" H 17050 10950 50  0001 C CNN
-F 3 "" H 17050 10950 50  0001 C CNN
-	1    17050 10950
+P 17050 10900
+F 0 "#PWR0103" H 17050 10750 50  0001 C CNN
+F 1 "+3V3" V 17065 11073 50  0000 C CNN
+F 2 "" H 17050 10900 50  0001 C CNN
+F 3 "" H 17050 10900 50  0001 C CNN
+	1    17050 10900
 	0    1    1    0
 $EndComp
 Wire Wire Line
-	16500 10950 17050 10950
+	16500 10900 17050 10900
 $Comp
 L power:+5V #PWR0104
 U 1 1 5BBD44FC
-P 17050 10850
-F 0 "#PWR0104" H 17050 10700 50  0001 C CNN
-F 1 "+5V" V 17065 10978 50  0000 L CNN
-F 2 "" H 17050 10850 50  0001 C CNN
-F 3 "" H 17050 10850 50  0001 C CNN
-	1    17050 10850
+P 17050 10800
+F 0 "#PWR0104" H 17050 10650 50  0001 C CNN
+F 1 "+5V" V 17065 10928 50  0000 L CNN
+F 2 "" H 17050 10800 50  0001 C CNN
+F 3 "" H 17050 10800 50  0001 C CNN
+	1    17050 10800
 	0    1    1    0
 $EndComp
 Wire Wire Line
-	16500 10850 17050 10850
+	16500 10800 17050 10800
 Wire Wire Line
 	950  4350 1450 4350
