File: OTTO-power/OTTO-power.sch (KiCad schematic (older format))
At the start: 45 parts, among them J1 Barrel_Jack, J2 Conn_01x10, J3 USB_B_Micro, J4 battery, SW1 SW_Push, SW2 SW_reset, U1 MAX8903A, U2 MAX17048, U3 TPS61090, U4 XC6210

Commit message: Revert "added a reset button to the power board"
This reverts commit bbfaa2fb8df27d7f63d1a584e9f51fc8f5fa6fe3.
Parts:
- removed R15: 1K, Resistor_SMD:R_0805_2012Metric, symbol Device:R_US
- removed SW2: SW_reset, Button_Switch_SMD:SW_SPST_B3U-3000P, symbol Switch:SW_Push
- C14: value 0.1uf -> 0.1uF
- C15: value 100uf -> 0.1uF
- J1: footprint Connector_BarrelJack:BarrelJack_CUI_PJ-102AH_Horizontal -> Connector_BarrelJack:BarrelJack_CUI_PJ-063AH_Horizontal
- R14: value 100K -> 10K
Connections:
- wire segments 186 -> 181
Changed lines of the file:
@@
 F 0 "J1" H 1850 6150 50  0000 R CNN
 F 1 "Barrel_Jack" H 2000 6050 50  0000 R CNN
-F 2 "Connector_BarrelJack:BarrelJack_CUI_PJ-102AH_Horizontal" H 1850 5810 50  0001 C CNN
+F 2 "Connector_BarrelJack:BarrelJack_CUI_PJ-063AH_Horizontal" H 1850 5810 50  0001 C CNN
 F 3 "~" H 1850 5810 50  0001 C CNN
 	1    1800 5850
@@
 	-1   0    0    1
 $EndComp
-Text GLabel 10450 5500 2    55   Input ~ 0
+Text GLabel 9800 5500 2    55   Input ~ 0
 EN_PI
 $Comp
@@
 AR Path="/5DEA7844/5BA9FC9D" Ref="C?"  Part="1"
 F 0 "C14" H 7692 5346 50  0000 L CNN
-F 1 "0.1uf" H 7692 5255 50  0000 L CNN
+F 1 "0.1uF" H 7692 5255 50  0000 L CNN
 F 2 "Capacitor_SMD:C_0805_2012Metric" H 7600 5300 50  0001 C CNN
 F 3 "~" H 7600 5300 50  0001 C CNN
@@
 AR Path="/5DEA7844/5BA9FCBF" Ref="R?"  Part="1"
 F 0 "R14" V 9000 5600 50  0000 L CNN
-F 1 "100K" V 9200 5600 50  0000 L CNN
+F 1 "10K" V 9200 5600 50  0000 L CNN
 F 2 "Resistor_SMD:R_0805_2012Metric" V 9140 5640 50  0001 C CNN
 F 3 "~" H 9100 5650 50  0001 C CNN
@@
 AR Path="/5DEA7844/5BA9FCCD" Ref="C?"  Part="1"
 F 0 "C15" V 8871 5900 50  0000 C CNN
-F 1 "100uf" V 8962 5900 50  0000 C CNN
+F 1 "0.1uF" V 8962 5900 50  0000 C CNN
 F 2 "Capacitor_SMD:C_0805_2012Metric" H 9100 5900 50  0001 C CNN
 F 3 "~" H 9100 5900 50  0001 C CNN
@@
 Connection ~ 9250 5650
 Wire Wire Line
-	8950 5500 9750 5500
+	8950 5500 9800 5500
 Text GLabel 3150 6150 2    55   Input ~ 0
 SENSE_PIN
@@
 Wire Wire Line
 	2750 3050 2750 3100
-$Comp
-L Switch:SW_Push SW2
-U 1 1 5BADCE51
-P 10100 5950
-F 0 "SW2" H 10100 6215 50  0000 C CNN
-F 1 "SW_reset" H 10100 6124 50  0000 C CNN
-F 2 "Button_Switch_SMD:SW_SPST_B3U-3000P" H 10100 6150 50  0001 C CNN
-F 3 "" H 10100 6150 50  0001 C CNN
-	1    10100 5950
-	-1   0    0    -1
-$EndComp
-Wire Wire Line
-	9900 5950 9750 5950
-Wire Wire Line
-	9750 5950 9750 5500
-Connection ~ 9750 5500
-Wire Wire Line
-	9750 5500 10450 5500
-$Comp
-L Device:R_US R15
-U 1 1 5BAEDA0F
-P 10450 5950
-AR Path="/5BAEDA0F" Ref="R15"  Part="1"
-AR Path="/5DEA7844/5BAEDA0F" Ref="R?"  Part="1"
-F 0 "R15" V 10350 5900 50  0000 L CNN
-F 1 "1K" V 10550 5900 50  0000 L CNN
-F 2 "Resistor_SMD:R_0805_2012Metric" V 10490 5940 50  0001 C CNN
-F 3 "~" H 10450 5950 50  0001 C CNN
-F 4 "-" H -16100 750 50  0001 C CNN "MFR"
-F 5 "-" H -16100 750 50  0001 C CNN "MPN"
-F 6 "-" H -16100 750 50  0001 C CNN "SPR"
-F 7 "-" H -16100 750 50  0001 C CNN "SPN"
-F 8 "-" H -16100 750 50  0001 C CNN "SPURL"
-	1    10450 5950
-	0    1    -1   0
-$EndComp
-Wire Wire Line
-	10750 5950 10750 6050
-$Comp
-L power:GNDREF #PWR0101
-U 1 1 5BAF631A
-P 10750 6050
-AR Path="/5BAF631A" Ref="#PWR0101"  Part="1"
-AR Path="/5DEA7844/5BAF631A" Ref="#PWR?"  Part="1"
-F 0 "#PWR0101" H 10750 5800 50  0001 C CNN
-F 1 "GNDREF" H 10755 5877 50  0001 C CNN
-F 2 "" H 10750 6050 50  0001 C CNN
-F 3 "" H 10750 6050 50  0001 C CNN
-	1    10750 6050
-	1    0    0    -1
-$EndComp
-Wire Wire Line
-	10750 5950 10600 5950
 $EndSCHEMATC

Commit message: Revert "Revert "added a reset button to the power board""
This reverts commit f20825db904c66ff1a5b44b22e19a70ce58abb56.
Parts:
- added R15: 1K, Resistor_SMD:R_0805_2012Metric, symbol Device:R_US
- added SW2: SW_reset, Button_Switch_SMD:SW_SPST_B3U-3000P, symbol Switch:SW_Push
- C14: value 0.1uF -> 0.1uf
- C15: value 0.1uF -> 100uf
- J1: footprint Connector_BarrelJack:BarrelJack_CUI_PJ-063AH_Horizontal -> Connector_BarrelJack:BarrelJack_CUI_PJ-102AH_Horizontal
- R14: value 10K -> 100K
Connections:
- wire segments 181 -> 186
Changed lines of the file:
@@
 F 0 "J1" H 1850 6150 50  0000 R CNN
 F 1 "Barrel_Jack" H 2000 6050 50  0000 R CNN
-F 2 "Connector_BarrelJack:BarrelJack_CUI_PJ-063AH_Horizontal" H 1850 5810 50  0001 C CNN
+F 2 "Connector_BarrelJack:BarrelJack_CUI_PJ-102AH_Horizontal" H 1850 5810 50  0001 C CNN
 F 3 "~" H 1850 5810 50  0001 C CNN
 	1    1800 5850
@@
 	-1   0    0    1
 $EndComp
-Text GLabel 9800 5500 2    55   Input ~ 0
+Text GLabel 10450 5500 2    55   Input ~ 0
 EN_PI
 $Comp
@@
 AR Path="/5DEA7844/5BA9FC9D" Ref="C?"  Part="1"
 F 0 "C14" H 7692 5346 50  0000 L CNN
-F 1 "0.1uF" H 7692 5255 50  0000 L CNN
+F 1 "0.1uf" H 7692 5255 50  0000 L CNN
 F 2 "Capacitor_SMD:C_0805_2012Metric" H 7600 5300 50  0001 C CNN
 F 3 "~" H 7600 5300 50  0001 C CNN
@@
 AR Path="/5DEA7844/5BA9FCBF" Ref="R?"  Part="1"
 F 0 "R14" V 9000 5600 50  0000 L CNN
-F 1 "10K" V 9200 5600 50  0000 L CNN
+F 1 "100K" V 9200 5600 50  0000 L CNN
 F 2 "Resistor_SMD:R_0805_2012Metric" V 9140 5640 50  0001 C CNN
 F 3 "~" H 9100 5650 50  0001 C CNN
@@
 AR Path="/5DEA7844/5BA9FCCD" Ref="C?"  Part="1"
 F 0 "C15" V 8871 5900 50  0000 C CNN
-F 1 "0.1uF" V 8962 5900 50  0000 C CNN
+F 1 "100uf" V 8962 5900 50  0000 C CNN
 F 2 "Capacitor_SMD:C_0805_2012Metric" H 9100 5900 50  0001 C CNN
 F 3 "~" H 9100 5900 50  0001 C CNN
@@
 Connection ~ 9250 5650
 Wire Wire Line
-	8950 5500 9800 5500
+	8950 5500 9750 5500
 Text GLabel 3150 6150 2    55   Input ~ 0
 SENSE_PIN
@@
 Wire Wire Line
 	2750 3050 2750 3100
+$Comp
+L Switch:SW_Push SW2
+U 1 1 5BADCE51
+P 10100 5950
+F 0 "SW2" H 10100 6215 50  0000 C CNN
+F 1 "SW_reset" H 10100 6124 50  0000 C CNN
+F 2 "Button_Switch_SMD:SW_SPST_B3U-3000P" H 10100 6150 50  0001 C CNN
+F 3 "" H 10100 6150 50  0001 C CNN
+	1    10100 5950
+	-1   0    0    -1
+$EndComp
+Wire Wire Line
+	9900 5950 9750 5950
+Wire Wire Line
+	9750 5950 9750 5500
+Connection ~ 9750 5500
+Wire Wire Line
+	9750 5500 10450 5500
+$Comp
+L Device:R_US R15
+U 1 1 5BAEDA0F
+P 10450 5950
+AR Path="/5BAEDA0F" Ref="R15"  Part="1"
+AR Path="/5DEA7844/5BAEDA0F" Ref="R?"  Part="1"
+F 0 "R15" V 10350 5900 50  0000 L CNN
+F 1 "1K" V 10550 5900 50  0000 L CNN
+F 2 "Resistor_SMD:R_0805_2012Metric" V 10490 5940 50  0001 C CNN
+F 3 "~" H 10450 5950 50  0001 C CNN
+F 4 "-" H -16100 750 50  0001 C CNN "MFR"
+F 5 "-" H -16100 750 50  0001 C CNN "MPN"
+F 6 "-" H -16100 750 50  0001 C CNN "SPR"
+F 7 "-" H -16100 750 50  0001 C CNN "SPN"
+F 8 "-" H -16100 750 50  0001 C CNN "SPURL"
+	1    10450 5950
+	0    1    -1   0
+$EndComp
+Wire Wire Line
+	10750 5950 10750 6050
+$Comp
+L power:GNDREF #PWR0101
+U 1 1 5BAF631A
+P 10750 6050
+AR Path="/5BAF631A" Ref="#PWR0101"  Part="1"
+AR Path="/5DEA7844/5BAF631A" Ref="#PWR?"  Part="1"
+F 0 "#PWR0101" H 10750 5800 50  0001 C CNN
+F 1 "GNDREF" H 10755 5877 50  0001 C CNN
+F 2 "" H 10750 6050 50  0001 C CNN
+F 3 "" H 10750 6050 50  0001 C CNN
+	1    10750 6050
+	1    0    0    -1
+$EndComp
+Wire Wire Line
+	10750 5950 10600 5950
 $EndSCHEMATC
