File: OTTO-power/OTTO-power.sch (KiCad schematic (older format))
At the start: 45 parts, among them J1 Barrel_Jack, J2 Conn_01x10, J3 USB_B_Micro, J4 battery, SW1 SW_Push, SW2 SW_reset, U1 MAX8903A, U2 MAX17048, U3 TPS61090, U4 XC6210

Commit message: progresses in the mainboard wiring
Changed lines of the file:
@@
 DOK_OUT
 Text GLabel 9800 5000 2    50   Input ~ 0
-BATT+
+SYS
 Wire Wire Line
 	9650 5000 9800 5000
@@
 	9200 1950 9200 2050
 Text GLabel 7950 850  1    50   Input ~ 0
-BATT+
+SYS
 Wire Wire Line
 	7950 850  7950 950

Commit message: added the OTTO-Keys board and fixed some of the mainboard issues
Parts:
- C215: renamed from C15; footprint Capacitor_SMD:C_0805_2012Metric -> Capacitor_SMD:C_1210_3225Metric
- renumbered C1 to C201, C9 to C202, C10 to C203, C2 to C204, C11 to C205, C12 to C206, C3 to C207, C4 to C208, C5 to C209, C6 to C210, C7 to C211, C13 to C212, C8 to C213, C14 to C214, D1 to D201, D2 to D202, D3 to D203, J1 to J201, J2 to J202, J3 to J203, J4 to J204, L2 to L201, L1 to L202, R1 to R201, R2 to R202, R7 to R203, R8 to R204, R3 to R205, R9 to R206, R4 to R207, R10 to R208, R11 to R209, R5 to R210, R6 to R211, R12 to R212, R13 to R213, R14 to R214, R15 to R215, SW1 to SW201, SW2 to SW202, U3 to U201, U1 to U202, U4 to U203, U2 to U204
