File: OTTO-dac/OTTOdac.sch (KiCad schematic (older format))
At the start: 38 parts, among them J1 Conn_01x10, J2 Audio_IN, J3 Audio_OUT, J4 SJ1-42536-SMT, J5 Speaker, U1 AMS1117-3.3, U2 SGTL5000, U3 LM4860, X1 XO32

Commit message: added the OTTO-Keys board and fixed some of the mainboard issues
Parts:
- C114: renamed from C11; footprint Capacitor_SMD:CP_Elec_5x4.5 -> Capacitor_SMD:CP_Elec_5x5.9
- C115: renamed from C13; footprint Capacitor_SMD:CP_Elec_5x4.5 -> Capacitor_SMD:CP_Elec_5x5.9
- renumbered C1 to C101, C2 to C102, C4 to C103, C7 to C104, C8 to C105, C6 to C106, C19 to C107, C3 to C108, C16 to C109, C15 to C110, C17 to C111, C14 to C112, C12 to C113, C18 to C116, C5 to C117, C10 to C118, C9 to C119, J4 to J101, J2 to J102, J3 to J103, J5 to J104, J1 to J105, L1 to L101, MK1 to MK101, R7 to R101, R8 to R102, R10 to R103, R5 to R104, R9 to R105, R6 to R106, R4 to R107, R3 to R108, U1 to U101, U2 to U102, U3 to U?, X1 to X101
